File: eswitch.kicad_pcb (KiCad board)
At the start: 4 copper layers, 181 x 57.5 mm, 153 parts, among them J1 Wuerth 691311400116, J2 +12V IN, J3 GND IN, J4 USB-C, J5 UART, SW1 RESET, SW2 BOOT, U1 BTS7008-1EPP, U10 ESP32-S3-WROOM-1-N8, U11 USBLC6-2SC6, U2 BTS7008-1EPP, U3 BTS7008-1EPP, U4 BTS7008-1EPP, U5 BTS7008-1EPP, U6 BTS7008-1EPP, U7 BTS7008-1EPP, U8 BTS7008-1EPP, U9 TPS54360B

Commit message: Routed board: DRC clean (0 copper violations, 0 unconnected), 3D models, KiCad 10 native format
- freerouting with temporary keep-outs, post-route prune/fix/stitch (tools/finish.py, tools/stitch.py)
- USB-C D+/D- pair tie-offs and VBUS on In2, CC2 hand-routed
- design rules and net classes persisted in eswitch.kicad_pro
- schematic and board upgraded to KiCad 10 file format

Co-Authored-By: Claude Fable 5.1 <noreply@anthropic.com>
Parts:
- turned J4 to 90 degrees
Routing:
- net GND: track 0.00 -> 285.6 mm, vias 0 -> 25
- net IN8: track 0.00 -> 230.8 mm, vias 0 -> 2
- net +3V3: track 0.00 -> 216.2 mm, vias 0 -> 9
- net DEN: track 0.00 -> 201.5 mm, vias 0 -> 10
- net IS8: track 0.00 -> 175.8 mm, vias 0 -> 2
- net IN7: track 0.00 -> 164.0 mm, vias 0 -> 3
- net IS6: track 0.00 -> 148.8 mm, vias 0 -> 2
- net IS7: track 0.00 -> 146.4 mm, vias 0 -> 3
- net IN6: track 0.00 -> 142.6 mm, vias 0 -> 3
- net IN5: track 0.00 -> 141.0 mm, vias 0 -> 3
- net IS4: track 0.00 -> 135.8 mm, vias 0 -> 3
- net IS5: track 0.00 -> 125.5 mm, vias 0 -> 3
- net IS2: track 0.00 -> 115.5 mm, vias 0 -> 4
- net IS3: track 0.00 -> 107.1 mm, vias 0 -> 4
- net IN4: track 0.00 -> 102.2 mm, vias 0 -> 3
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