File: eswitch.kicad_pcb (KiCad board)
At the start: 4 copper layers, 221 x 75 mm, 194 parts, among them J1 691218410002, J10 691218410002, J11 691218410002, J12 691218410002, J2 BATT+ 9-16V, J3 GND IN, J4 USB-C, J5 UART, J6 691218410002, J7 691218410002, J8 691218410002, J9 691218410002, Q1 BSC016N06NS, Q2 BSC016N06NS, Q3 BSC016N06NS, Q4 BSC016N06NS, Q5 BSC016N06NS, SW1 RESET, SW2 BOOT, U1 BTS7004-1EPP, U10 ESP32-S3-WROOM-1-N8, U11 SRV05-4HTG-D, U12 LM74800-Q1, U13 LM74800-Q1, U2 BTS7004-1EPP, U3 BTS7008-1EPR, U4 BTS7008-1EPR, U5 BTS7008-1EPR, U6 BTS7008-1EPR, U7 BTS7008-1EPR, U8 BTS7002-1EPP, U9 TPSM63603V3

Commit message: Release revision B for prototype fabrication
Complete the routed PCB, capacitor correction, startup and SOA screening, and owner-confirmed physical-fit review. Include the verified fabrication package, three-board BOM, release gates, and controlled bring-up plan. Keep production qualification and the measured 40 A rating pending hardware validation.
Parts:
- added D7: STPS41L60CG, Package_TO_SOT_SMD:TO-263-2, B.Cu at (113.0, 40.0)
- added R17: 8.25k 1%, Resistor_SMD:R_0603_1608Metric, B.Cu at (89.0, 42.0)
- added R18: 1k, Resistor_SMD:R_0603_1608Metric, B.Cu at (89.0, 45.2)
- added R19: 10R, Resistor_SMD:R_0603_1608Metric, B.Cu at (100.5, 20.0)
- added R20: 1mR 1% 4W, eswitch:Bourns_CSS4J_4026, B.Cu at (74.0, 17.3)
- added U14: TPS2492 (LATCH), Package_SO:TSSOP-14_4.4x5mm_P0.65mm, B.Cu at (84.5, 34.5)
- C12, C13, C7, C8: value 22uF 10V -> 47uF 6.3V X7R
- C18: value 10nF 50V -> 10nF 50V C0G 5%
- J2: value BATT+ 9-16V -> BATT+ 9.5-16V
- Q3, Q4: value BSC016N06NS -> PSMN1R8-80SSE; footprint Package_SON:Infineon_PG-TDSON-8_6.15x5.15mm -> Package_TO_SOT_SMD:LFPAK88
- R12: value 127k 0.1% -> 115k 0.1%
- R14: value 59k 0.1% -> 56.2k 0.1%
- R16: value 100R -> 10R
- U10: footprint RF_Module:ESP32-S3-WROOM-1 -> eswitch:ESP32-S3-WROOM-1_Edge
- moved R15 40.1 mm to (93.0, 41.5), turned to 0 degrees
- moved R16 39.7 mm to (100.5, 7.00), turned to 180 degrees
- moved R14 36.4 mm to (93.0, 38.5), turned to 180 degrees
- moved C201 32.0 mm to (139.9, 34.6)
- moved C304 32.0 mm to (158.8, 39.0)
- moved D101 32.0 mm to (128.0, 51.5)
- moved F2 32.0 mm to (145.9, 17.5)
- moved J6 32.0 mm to (142.1, 69.8)
- moved R108 32.0 mm to (128.0, 55.0)
- moved R301 32.0 mm to (157.3, 43.0)
- moved R302 32.0 mm to (157.3, 46.2)
- moved U2 32.0 mm to (145.9, 35.0)
- moved C101 32.0 mm to (124.6, 34.6)
- moved C102 32.0 mm to (130.8, 42.5)
- moved C103 32.0 mm to (124.4, 49.2)
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Connections:
- C18 pad 1: /SLEW_MAIN -> /HS_TIMER
- Q3 pad 1: +12V -> /GATE_Q3
- Q3 pad 4: /HGATE_MAIN -> +12V
- Q3 pad 5: /BATT_MID -> /BATT_SENSE
- Q4 pad 1: +12V -> /GATE_Q4
- Q4 pad 4: /HGATE_MAIN -> +12V
- Q4 pad 5: /BATT_MID -> /BATT_SENSE
- R12 pad 1: /OV_TOP -> /BATT_MID
- R14 pad 1: /BATT_RAW -> /BATT_MID
- R16 pad 2: /SLEW_MAIN -> /GATE_Q3
- U12 pad 3: /BATT_RAW -> /BATT_MID
- U12 pad 4: /OV_TOP -> /BATT_MID
- U12 pad 5: /OV_MAIN -> GND
- U12 pad 6: /UV_MAIN -> /BATT_RAW
- U12 pad 8: /HGATE_MAIN -> (no net)
- U12 pad 9: +12V -> /BATT_MID
Routing:
- net /IN3: track 4.81 -> 184.0 mm, vias 1 -> 8
- net /INR2: track 19.9 -> 119.0 mm, vias 2 -> 5
- net /BATT_MID: track 19.4 -> 74.5 mm, vias 28 -> 30
- net /IS1: track 128.8 -> 171.1 mm, vias 2 -> 4
- net +12V: track 17.2 -> 56.0 mm, vias 13 -> 26
- net /IS3: track 145.3 -> 183.1 mm, vias 2 -> 4
- net /IN2: track 136.6 -> 172.6 mm, vias 4 -> 6
- net /IS8: track 216.3 -> 252.1 mm, vias 5 -> 6
- net /IN5: track 171.4 -> 206.1 mm, vias 5 -> 7
- net /IS2: track 122.4 -> 155.4 mm, vias 4 -> 6
- net /DEN: track 319.0 -> 351.6 mm, vias 12 -> 14
- net /IN7: track 202.4 -> 235.0 mm
- net /IN6: track 234.9 -> 267.1 mm
- net +3V3: track 330.7 -> 362.9 mm, vias 21 -> 19
- net /IS4: track 195.7 -> 227.7 mm
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- added copper zone on B.Cu, net /BATT_SENSE
- added copper zone on F.Cu, net /BATT_SENSE
- added copper zone on In2.Cu, net /BATT_SENSE
Other:
- board size 221 x 75 mm -> 253 x 75 mm
- board text added: "BATT+ 9.5-16V"
- board text added: "FAULT: CYCLE BATTERY"
- board text removed: "BATT+ 9-16V"
