File: eswitch.kicad_sch (KiCad schematic)
At the start: 153 parts, among them J1 Wuerth 691311400116, J2 +12V IN, J3 GND IN, J4 USB-C, J5 UART, SW1 RESET, SW2 BOOT, U1 BTS7004-1EPP, U10 ESP32-S3-WROOM-1-N8, U11 USBLC6-2SC6, U2 BTS7004-1EPP, U3 BTS7008-1EPP, U4 BTS7008-1EPP, U5 BTS7008-1EPP, U6 BTS7008-1EPP, U7 BTS7008-1EPP, U8 BTS7002-1EPP, U9 TPS54360B

Commit message: Apply review corrections and circuit/fuse silk; hold fabrication
Add dated three-board DigiKey BOM for manual assembly, direct-entry outputs and higher-current input terminals. Mark each fuse with circuit identity and maximum fuse size. Preserve legacy fabrication files in a do-not-order archive and gate new outputs on release checks.

Not order-ready: eight signal connections remain after input terminal migration; native parity and electrical/layout/thermal findings are documented in docs/critical-review.md.
Parts:
- removed J3: GND IN, eswitch:ScrewTerminal_Keystone_8196_10-32, symbol Connector:Screw_Terminal_01x01
- added H4: M3, MountingHole:MountingHole_3.2mm_M3, symbol Mechanical:MountingHole
- added J10, J11, J6, J7, J8, J9: 691218410002, eswitch:TerminalBlock_1x02_P7.62mm_Wuerth_2184, symbol Connector:Screw_Terminal_01x02
- added J2: +12V IN, eswitch:ScrewTerminal_Wuerth_74650195_M5, symbol Connector:Screw_Terminal_01x01
- C10, C3, C4: MPN CL10B104KB8NNNC -> CC0603KRX7R9BB104; Manufacturer Samsung Electro-Mechanics -> YAGEO
- C103, C203, C303, C403, C503, C603, C703, C803: MPN CL10C221JB8NNNC -> CL10C221JB8NFNC
- C11: MPN CL10B105KO8NNNC -> CC0603KRX7R7BB105; Manufacturer Samsung Electro-Mechanics -> YAGEO
- C5: MPN CL10B273KB8NNNC -> CC0603KRX7R9BB273; Manufacturer Samsung Electro-Mechanics -> YAGEO
- C9: MPN CL21A106KPFNNNE -> CC0805KKX5R6BB106; Manufacturer Samsung Electro-Mechanics -> YAGEO
- D1, D4: value SS36 -> B360A; MPN B360-13-F -> B360A-13-F
- D101, D201, D301, D401, D501, D601, D701, D801: MPN BAT54S,215 -> BAT54S-QR
- D2: value SS36 -> B360A; MPN B360-13-F -> B360A-13-F; Note USB -> VIN -> USB -> VIN; low-VBUS margin unresolved
- J1: value Wuerth 691311400116 -> 691218410002; footprint eswitch:TerminalBlock_1x16_P7.62mm_Wuerth_3114 -> eswitch:TerminalBlock_1x02_P7.62mm_Wuerth_2184; symbol Connector:Screw_Terminal_01x16 -> Connector:Screw_Terminal_01x02; MPN 691311400116 -> 691218410002; Note odd pins = GND, even pins = LOAD+ -> CH1: pin 1 GND, pin 2 LOAD+; direct-entry screw clamp; 30 A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
- J12: renamed from J2; value +12V IN -> 691218410002; footprint eswitch:ScrewTerminal_Keystone_8196_10-32 -> eswitch:TerminalBlock_1x02_P7.62mm_Wuerth_2184; symbol Connector:Screw_Terminal_01x01 -> Connector:Screw_Terminal_01x02; MPN 8196 -> 691218410002; Manufacturer Keystone Electronics -> Wurth Elektronik; Note (none) -> CH8: pin 1 GND, pin 2 LOAD+; direct-entry screw clamp; 30 A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
- J3: renamed from H4; value M3 -> GND IN; footprint MountingHole:MountingHole_3.2mm_M3 -> eswitch:ScrewTerminal_Wuerth_74650195_M5; symbol Mechanical:MountingHole -> Connector:Screw_Terminal_01x01; MPN (none) -> 74650195; Manufacturer (none) -> Wurth Elektronik; Note (none) -> M5 ring-lug terminal, 85 A at 20 C component rating; PCB/wi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
- R1: MPN RC0603FR-07200KL -> ERJ-3EKF2003V; Manufacturer YAGEO -> Panasonic
- R107, R207, R307, R407, R507, R607, R707, R807: value 2.2k -> 10k; MPN RC0603FR-072K2L -> RC0603FR-0710KL; Note RLED -> RLED; <=78.4 mW at 28 V even with LED shorted
- R7, R8: MPN RC0603FR-075K1L -> ERJ-3EKF5101V; Manufacturer YAGEO -> Panasonic
- SW1, SW2: MPN PTS645SM43SMTR92 -> PTS645SM43SMTR92 LFS
- U11: value USBLC6-2SC6 -> SRV05-4HTG-D; symbol Power_Protection:USBLC6-2P6 -> Power_Protection:SRV05-4; MPN USBLC6-2SC6 -> SRV05-4HTG-D; Manufacturer STMicroelectronics -> Littelfuse; Note (none) -> Four independent steering channels; pair 1+6 and 3+4 extern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
- U3, U4, U5, U6, U7: value BTS7008-1EPP -> BTS7008-1EPR; symbol eswitch:BTS7008-1EPP -> eswitch:BTS7008-1EPR
Connections:
- net +12V: now also J2.1 (Pin_1); no longer J12.1 (Pin_1)
- net GND: now also J12.1 (Pin_1), J3.1 (Pin_1), J10.1 (Pin_1), J11.1 (Pin_1), J6.1 (Pin_1), J7.1 (Pin_1), J8.1 (Pin_1), J9.1 (Pin_1); no longer J1.11 (Pin_11), J1.13 (Pin_13), J1.15 (Pin_15), J1.3 (Pin_3), J1.5 (Pin_5), J1.7 (Pin_7), J1.9 (Pin_9)
- net LOAD2: now also J6.2 (Pin_2); no longer J1.4 (Pin_4)
- net LOAD3: now also J7.2 (Pin_2); no longer J1.6 (Pin_6)
- net LOAD4: now also J8.2 (Pin_2); no longer J1.8 (Pin_8)
- net LOAD5: now also J9.2 (Pin_2); no longer J1.10 (Pin_10)
- net LOAD6: now also J10.2 (Pin_2); no longer J1.12 (Pin_12)
- net LOAD7: now also J11.2 (Pin_2); no longer J1.14 (Pin_14)
- net LOAD8: now also J12.2 (Pin_2); no longer J1.16 (Pin_16)
Other:
- note added: "8-channel PROFET+2 12 V load switch with 3-position ATO fuse bypass"
- note added: "I/O: J1, J6-J12 direct-entry load terminals: pin 1=GND, pin 2=LOAD+"
- note added: "SUPPLY: boat house battery via battery-side feeder fuse; DC-DC charging; input protection under review"
- note removed: "8-channel PROFET+2 (BTS7008-1EPP) 12 V load switch with 3-position ATO fuse bypass"
- note removed: "I/O: J1 load terminals (odd=LOAD+, even=GND), J2/J3 #10 screw terminals"

Commit message: Finish reviewed PCB routing and release checks
Parts:
- C10, C3, C4: MPN CC0603KRX7R9BB104 -> CC0603JRX7R9BB104
- H1, H2, H3, H4: now left out of the parts list
Changed lines of the file:
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@@
 			)
 		)
-		(property "MPN" "CC0603KRX7R9BB104"
+		(property "MPN" "CC0603JRX7R9BB104"
 			(at 345.44 125.73 0)
 			(effects
@@
 			)
 		)
-		(property "MPN" "CC0603KRX7R9BB104"
+		(property "MPN" "CC0603JRX7R9BB104"
 			(at 396.24 240.03 0)
 			(effects
@@
 			)
 		)
-		(property "MPN" "CC0603KRX7R9BB104"
+		(property "MPN" "CC0603JRX7R9BB104"
 			(at 393.7 274.32 0)
 			(effects
@@
 		(unit 1)
 		(exclude_from_sim no)
-		(in_bom yes)
+		(in_bom no)
 		(on_board yes)
 		(dnp no)
@@
 		(unit 1)
 		(exclude_from_sim no)
-		(in_bom yes)
+		(in_bom no)
 		(on_board yes)
 		(dnp no)
@@
 		(unit 1)
 		(exclude_from_sim no)
-		(in_bom yes)
+		(in_bom no)
 		(on_board yes)
 		(dnp no)
@@
 		(unit 1)
 		(exclude_from_sim no)
-		(in_bom yes)
+		(in_bom no)
 		(on_board yes)
 		(dnp no)

Commit message: Checkpoint unfinished revision B power protection and PCB review
Parts:
- removed C1: 4.7uF 50V, Capacitor_SMD:C_1210_3225Metric, symbol Device:C
- removed C4: 100nF 25V, Capacitor_SMD:C_0603_1608Metric, symbol Device:C
- removed C5: 27nF, Capacitor_SMD:C_0603_1608Metric, symbol Device:C
- removed C6: 150pF, Capacitor_SMD:C_0603_1608Metric, symbol Device:C
- removed D4: B360A, Diode_SMD:D_SMA, symbol Device:D_Schottky
- removed J12: 691218410002, eswitch:TerminalBlock_1x02_P7.62mm_Wuerth_2184, symbol Connector:Screw_Terminal_01x02
- removed J2: +12V IN, eswitch:ScrewTerminal_Wuerth_74650195_M5, symbol Connector:Screw_Terminal_01x01
- removed L1: 10uH 4A, Inductor_SMD:L_Bourns_SRP7028A_7.3x6.6mm, symbol Device:L
- removed R2: 31.6k 1%, Resistor_SMD:R_0603_1608Metric, symbol Device:R
- removed R3: 10.2k 1%, Resistor_SMD:R_0603_1608Metric, symbol Device:R
- removed R4: 3.9k, Resistor_SMD:R_0603_1608Metric, symbol Device:R
- removed U9: TPS54360B, Package_SO:TI_SO-PowerPAD-8_ThermalVias, symbol Regulator_Switching:TPS54360DDA
- added C104, C204, C304, C404, C504, C604, C704, C804: 47nF 50V, Capacitor_SMD:C_0805_2012Metric, symbol Device:C
- added C12, C13: 22uF 10V, Capacitor_SMD:C_1210_3225Metric, symbol Device:C
- added C14: 1uF, Capacitor_SMD:C_0603_1608Metric, symbol Device:C
- added C15, C16, C19, C20, C21: 100nF 50V, Capacitor_SMD:C_0805_2012Metric, symbol Device:C
- added C17, C22: 4.7uF 50V, Capacitor_SMD:C_1210_3225Metric, symbol Device:C
- added C18: 10nF 50V C0G 5%, Capacitor_SMD:C_0805_2012Metric, symbol Device:C
- added D6: SMCJ16A, Diode_SMD:D_SMC, symbol Device:D_Zener
- added D7: STPS41L60CG, Package_TO_SOT_SMD:TO-263-2, symbol eswitch:STPS41L60C
- added J1, J6: 691218410002, eswitch:TerminalBlock_1x02_P7.62mm_Wuerth_2184, symbol Connector:Screw_Terminal_01x02
- added NT1: AGND STAR, NetTie:NetTie-2_SMD_Pad0.5mm, symbol Device:NetTie_2
- added Q1, Q2, Q5: BSC016N06NS, Package_SON:Infineon_PG-TDSON-8_6.15x5.15mm, symbol eswitch:BSC016N06NS
- added Q3, Q4: PSMN1R8-80SSE, Package_TO_SOT_SMD:LFPAK88, symbol eswitch:PSMN1R8-80SSE
- added R10, R11: 22R, Resistor_SMD:R_0603_1608Metric, symbol Device:R
- added R108, R208, R308, R408, R508, R608, R708, R808: 47k, Resistor_SMD:R_0603_1608Metric, symbol Device:R
- added R12: 115k 0.1%, Resistor_SMD:R_0603_1608Metric, symbol Device:R
- added R13, R15: 10k 0.1%, Resistor_SMD:R_0603_1608Metric, symbol Device:R
- added R14: 56.2k 0.1%, Resistor_SMD:R_0603_1608Metric, symbol Device:R
- added R16, R19: 10R, Resistor_SMD:R_0603_1608Metric, symbol Device:R
- added R17: 8.25k 1%, Resistor_SMD:R_0603_1608Metric, symbol Device:R
- added R18: 1k, Resistor_SMD:R_0603_1608Metric, symbol Device:R
- added R20: 1mR 1% 4W, eswitch:Bourns_CSS4J_4026, symbol eswitch:Kelvin_Shunt
- added U12, U13: LM74800-Q1, Package_SON:WSON-12-1EP_3x3mm_P0.5mm_EP1.5x2.5mm, symbol eswitch:LM74800
- added U14: TPS2492 (LATCH), Package_SO:TSSOP-14_4.4x5mm_P0.65mm, symbol eswitch:TPS2492
- added U9: TPSM63603V3, eswitch:TI_RDH0030A_TPSM63603, symbol eswitch:TPSM63603V3
- C1: renamed from D3; value SMBJ26A -> 4.7uF 50V; footprint Diode_SMD:D_SMB -> Capacitor_SMD:C_1210_3225Metric; symbol Device:D_Zener -> Device:C; MPN SMBJ26A -> GRM32ER71H475KA88L; Manufacturer Littelfuse -> Murata; Note bus TVS -> (none)
- D3: renamed from D2; value B360A -> SMCJ24CA; footprint Diode_SMD:D_SMA -> Diode_SMD:D_SMC; symbol Device:D_Schottky -> Device:D_Zener; MPN B360A-13-F -> SMCJ24CA; Manufacturer Diodes Incorporated -> Littelfuse; Note USB -> VIN; low-VBUS margin unresolved -> Bidirectional input clamp; upstream fuse required
- J10: renamed from J8; Note CH4: pin 1 GND, pin 2 LOAD+; direct-entry screw clamp; 30 A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 -> CH6: pin 1 GND, pin 2 LOAD+; direct-entry screw clamp; 30 A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
- J11: renamed from J9; Note CH5: pin 1 GND, pin 2 LOAD+; direct-entry screw clamp; 30 A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 -> CH7: pin 1 GND, pin 2 LOAD+; direct-entry screw clamp; 30 A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
- J12: renamed from J10; Note CH6: pin 1 GND, pin 2 LOAD+; direct-entry screw clamp; 30 A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 -> CH8: pin 1 GND, pin 2 LOAD+; direct-entry screw clamp; 30 A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
- J2: renamed from J11; value 691218410002 -> BATT+ 9.5-16V; footprint eswitch:TerminalBlock_1x02_P7.62mm_Wuerth_2184 -> eswitch:ScrewTerminal_Wuerth_74650195_M5; symbol Connector:Screw_Terminal_01x02 -> Connector:Screw_Terminal_01x01; MPN 691218410002 -> 74650195; Note CH7: pin 1 GND, pin 2 LOAD+; direct-entry screw clamp; 30 A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 -> M5 ring-lug terminal, 85 A at 20 C component rating; PCB/wi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
- J7: renamed from J1; Note CH1: pin 1 GND, pin 2 LOAD+; direct-entry screw clamp; 30 A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 -> CH3: pin 1 GND, pin 2 LOAD+; direct-entry screw clamp; 30 A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
- J8: renamed from J6; Note CH2: pin 1 GND, pin 2 LOAD+; direct-entry screw clamp; 30 A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 -> CH4: pin 1 GND, pin 2 LOAD+; direct-entry screw clamp; 30 A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
- J9: renamed from J7; Note CH3: pin 1 GND, pin 2 LOAD+; direct-entry screw clamp; 30 A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 -> CH5: pin 1 GND, pin 2 LOAD+; direct-entry screw clamp; 30 A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
- R1: value 200k 1% -> 16.5k 1%; MPN ERJ-3EKF2003V -> RC0603FR-0716K5L; Manufacturer Panasonic -> YAGEO; Note fsw 500 kHz -> 800 kHz per TPSM63603 table 7-4
- U11: Note Four independent steering channels; pair 1+6 and 3+4 extern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 -> ESD at USB connector; pair 1+6 and 3+4; pin 2 GND, pin 5 VB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
Connections:
- net +12V: now also C19.1, D6.1 (K), D7.2 (K_TAB), Q3.2 (S), Q3.3 (S), Q3.4 (S), Q4.2 (S), Q4.3 (S), Q4.4 (S), U14.11 (OUT); no longer C1.1 (K)
- net +3V3: now also C12.1, C13.1, U9.10 (VOUT), U9.12 (VOUT), U9.13 (VOUT), U9.14 (VOUT), U9.15 (VOUT), U9.22 (VLDOIN), U9.25 (FB), U9.30 (VOUT), U9.7 (VOUT), U9.8 (VOUT), U9.9 (VOUT)
- net GND: now also D3.2 (A), C12.2, C13.2, C14.2, C15.2, C16.2, C18.2, C19.2, C20.2, C21.2, D6.2 (A), D7.1 (A1), D7.3 (A2), J1.1 (Pin_1), J6.1 (Pin_1), NT1.2, R13.2, R15.2, R18.2, U12.5 (OV), U12.7 (GND), U13.5 (OV), U13.7 (GND), U14.7 (GND), U9.16 (PGND), U9.17 (PGND), U9.28 (PGND), U9.29 (PGND), U9.5 (PGND), U9.6 (PGND); no longer J2.1 (Pin_1), R1.2
- net INR1: now also R108.1
- net INR2: now also R208.1
- net INR3: now also R308.1
- net INR4: now also R408.1
- net INR5: now also R508.1
- net INR6: now also R608.1
- net INR7: now also R708.1
- net INR8: now also R808.1
- net LOAD1: now also J1.2 (Pin_2); no longer J7.2 (Pin_2)
- net LOAD2: now also J6.2 (Pin_2); no longer J8.2 (Pin_2)
- net LOAD3: now also J7.2 (Pin_2); no longer J9.2 (Pin_2)
- net LOAD4: now also J8.2 (Pin_2); no longer J10.2 (Pin_2)
- net LOAD5: now also J9.2 (Pin_2); no longer J11.2 (Pin_2)
- net LOAD6: now also J10.2 (Pin_2); no longer J12.2 (Pin_2)
- net LOAD7: now also J11.2 (Pin_2); no longer J2.2 (Pin_2)
- net LOAD8: now also J12.2 (Pin_2)
- net RT: now also U9.1 (RT)
- net UGND1: now also C104.2, R108.2
- net UGND2: now also C204.2, R208.2
- net UGND3: now also C304.2, R308.2
- net UGND4: now also C404.2, R408.2
- net UGND5: now also C504.2, R508.2
- net UGND6: now also C604.2, R608.2
- net UGND7: now also C704.2, R708.2
- net UGND8: now also C804.2, R808.2
- net USB_D+: now also R10.1; no longer U10.14 (USB_D+)
- net USB_D-: now also R11.1; no longer U10.13 (USB_D-)
- net VBUS: now also C20.1, Q5.1 (S), Q5.2 (S), Q5.3 (S), U13.2 (A), U13.6 (EN/UVLO); no longer D3.2 (A)
- net VIN: now also C1.1, C21.1, C22.2, Q5.5 (D), U13.10 (VS), U13.12 (C), U13.3 (VSNS), U13.4 (SW), U13.9 (OUT), U9.18 (VIN), U9.19 (VIN), U9.2 (EN/SYNC), U9.3 (VIN), U9.4 (VIN); no longer D3.1 (K)
- net VS1: now also C104.1
- net VS2: now also C204.1
- net VS3: now also C304.1
- net VS4: now also C404.1
- net VS5: now also C504.1
- net VS6: now also C604.1
- net VS7: now also C704.1
- net VS8: now also C804.1
- new net AGND_BUCK: NT1.1, R1.2, U9.24 (AGND), U9.27 (AGND)
- new net BATT_MID: C16.1, C17.2, Q1.5 (D), Q2.5 (D), R12.1, R14.1, R20.1 (I_IN), U12.10 (VS), U12.12 (C), U12.3 (VSNS), U12.4 (SW), U12.9 (OUT)
- new net BATT_RAW: C15.1, D3.1 (K), J2.1 (Pin_1), Q1.1 (S), Q1.2 (S), Q1.3 (S), Q2.1 (S), Q2.2 (S), Q2.3 (S), U12.2 (A), U12.6 (EN/UVLO)
- new net BATT_SENSE: Q3.5 (D_MB), Q4.5 (D_MB), R20.2 (I_OUT)
- new net CAP_MAIN: C17.1, U12.11 (CAP)
- new net CAP_USB: C22.1, U13.11 (CAP)
- new net DGATE_MAIN: Q1.4 (G), Q2.4 (G), U12.1 (DGATE)
- new net DGATE_USB: Q5.4 (G), U13.1 (DGATE)
- new net GATE_Q3: Q3.1 (G), R16.2
- new net GATE_Q4: Q4.1 (G), R19.2
- new net HGATE_MAIN: R16.1, R19.1, U14.12 (GATE)
- new net HS_PROG: R17.2, R18.1, U14.3 (PROG)
- new net HS_REF: R17.1, U14.2 (VREF)
- new net HS_SENSE: R20.4 (S_OUT), U14.13 (SENSE)
- new net HS_TIMER: C18.1, U14.4 (TIMER)
- new net HS_VCC: R20.3 (S_IN), U14.14 (VCC)
- new net OV_MAIN: R12.2, R13.1, U14.5 (OV)
- new net USB_MCU_D+: R10.2, U10.14 (USB_D+)
- new net USB_MCU_D-: R11.2, U10.13 (USB_D-)
- new net UV_MAIN: R14.2, R15.1, U14.1 (UVEN)
- new net VCC_BUCK: C14.1, U9.23 (VCC)
- no-connect marks 16 -> 23
Other:
- note added: "INPUT: 9.5-16V; U12 reverse block; U14 current/power limit + latch-off; U12/U13 RTN FLOAT"
- note added: "LOGIC: protected +12V -> F9 -> D1 -> VIN; USB -> Q5 ideal diode -> VIN; TPSM63603V3 -> 3V3"
- note added: "SUPPLY: 9.5-16V house bank via upstream fuse; USB initial programming only, battery disconnected"
- note removed: "POWER: +12V -> F9 -> D1 -> VIN <- D2 <- USB VBUS; TPS54360B 500 kHz buck -> +3V3"
- note removed: "SUPPLY: boat house battery via battery-side feeder fuse; DC-DC charging; input protection under review"
- moved on the sheet: D3, J10, J11, J12, J7, J8, J9

Commit message: Release revision B for prototype fabrication
Complete the routed PCB, capacitor correction, startup and SOA screening, and owner-confirmed physical-fit review. Include the verified fabrication package, three-board BOM, release gates, and controlled bring-up plan. Keep production qualification and the measured 40 A rating pending hardware validation.
Parts:
- C12, C13, C7, C8: value 22uF 10V -> 47uF 6.3V X7R; MPN GRM32ER71A226KE20L -> GCM32ER70J476KE19L
- U10: footprint RF_Module:ESP32-S3-WROOM-1 -> eswitch:ESP32-S3-WROOM-1_Edge
Changed lines of the file:
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@@
 			)
 		)
-		(property "Footprint" "RF_Module:ESP32-S3-WROOM-1"
+		(property "Footprint" "eswitch:ESP32-S3-WROOM-1_Edge"
 			(at 381 80.01 0)
 			(effects
@@
 			)
 		)
-		(property "Value" "22uF 10V"
+		(property "Value" "47uF 6.3V X7R"
 			(at 386.715 302.26 0)
 			(effects
@@
 			)
 		)
-		(property "MPN" "GRM32ER71A226KE20L"
+		(property "MPN" "GCM32ER70J476KE19L"
 			(at 386.08 299.72 0)
 			(effects
@@
 			)
 		)
-		(property "Value" "22uF 10V"
+		(property "Value" "47uF 6.3V X7R"
 			(at 396.875 302.26 0)
 			(effects
@@
 			)
 		)
-		(property "MPN" "GRM32ER71A226KE20L"
+		(property "MPN" "GCM32ER70J476KE19L"
 			(at 396.24 299.72 0)
 			(effects
@@
 			)
 		)
-		(property "Value" "22uF 10V"
+		(property "Value" "47uF 6.3V X7R"
 			(at 417.195 302.26 0)
 			(effects
@@
 			)
 		)
-		(property "MPN" "GRM32ER71A226KE20L"
+		(property "MPN" "GCM32ER70J476KE19L"
 			(at 416.56 299.72 0)
 			(effects
@@
 			)
 		)
-		(property "Value" "22uF 10V"
+		(property "Value" "47uF 6.3V X7R"
 			(at 427.355 302.26 0)
 			(effects
@@
 			)
 		)
-		(property "MPN" "GRM32ER71A226KE20L"
+		(property "MPN" "GCM32ER70J476KE19L"
 			(at 426.72 299.72 0)
 			(effects
