File: eswitch.kicad_sch (KiCad schematic)
At the start: 200 parts, among them J1 691218410002, J10 691218410002, J11 691218410002, J12 691218410002, J2 BATT+ 9.5-16V, J3 GND IN, J4 USB-C, J5 UART, J6 691218410002, J7 691218410002, J8 691218410002, J9 691218410002, Q1 BSC016N06NS, Q2 BSC016N06NS, Q3 PSMN1R8-80SSE, Q4 PSMN1R8-80SSE, Q5 BSC016N06NS, SW1 RESET, SW2 BOOT, U1 BTS7004-1EPP, U10 ESP32-S3-WROOM-1-N8, U11 SRV05-4HTG-D, U12 LM74800-Q1, U13 LM74800-Q1, U14 TPS2492 (LATCH), U2 BTS7004-1EPP, U3 BTS7008-1EPR, U4 BTS7008-1EPR, U5 BTS7008-1EPR, U6 BTS7008-1EPR, U7 BTS7008-1EPR, U8 BTS7002-1EPP, U9 TPSM63603V3

Commit message: Release revision C with independent channel protection
Add hardware fault isolation for every AUTO and BYPASS output, complete the layout corrections, and update monitoring and bring-up documentation.

Include verified prototype fabrication packages, CAM and JLC upload evidence, and per-unit BOM pricing. ERC, DRC, routing and schematic parity are clean; 29 transient cases pass.
Parts:
- removed C22: 4.7uF 50V, Capacitor_SMD:C_1210_3225Metric, symbol Device:C
- removed J12: 691218410002, eswitch:TerminalBlock_1x02_P7.62mm_Wuerth_2184, symbol Connector:Screw_Terminal_01x02
- removed J2: BATT+ 9.5-16V, eswitch:ScrewTerminal_Wuerth_74650195_M5, symbol Connector:Screw_Terminal_01x01
- removed R108: 47k, Resistor_SMD:R_0603_1608Metric, symbol Device:R
- removed R16: 10R, Resistor_SMD:R_0603_1608Metric, symbol Device:R
- added C111, C112, C211, C212, C311, C312, C411, C412, C511, C512, C611, C612, C711, C712, C811, C812: 100nF 50V U2J 5%, Capacitor_SMD:C_1206_3216Metric, symbol Device:C
- added C113, C213, C313, C413, C513, C613, C713, C813: 100nF 50V, Capacitor_SMD:C_0805_2012Metric, symbol Device:C
- added C114, C115, C116, C214, C215, C216, C314, C315, C316, C414, C415, C416, C514, C515, C516, C614, C615, C616, C714, C715, C716, C814, C815, C816: 120uF 35V polymer, Capacitor_SMD:CP_Elec_10x12.6, symbol Device:C_Polarized
- added C23, C24: 10nF 50V, Capacitor_SMD:C_0805_2012Metric, symbol Device:C
- added C25, C28: 12nF 50V C0G 5%, Capacitor_SMD:C_0805_2012Metric, symbol Device:C
- added C804: 47nF 50V, Capacitor_SMD:C_0805_2012Metric, symbol Device:C
- added D103, D112, D203, D212, D303, D312, D403, D412, D503, D512, D603, D612, D703, D712, D8, D803, D812, D9: BAT54S, Package_TO_SOT_SMD:SOT-23, symbol Diode:BAT54S
- added D111, D211, D311, D411, D511, D611, D711, D811: STPS41L60CG, Package_TO_SOT_SMD:TO-263-2, symbol eswitch:STPS41L60C
- added H10, H11, H12, H4, H5, H6, H7, H8, H9: M3, MountingHole:MountingHole_3.2mm_M3, symbol Mechanical:MountingHole
- added J3: GND IN, eswitch:ScrewTerminal_Wuerth_74650195_M5, symbol Connector:Screw_Terminal_01x01
- added Q11, Q12, Q13, Q14, Q15, Q16, Q17, Q18: PSMN1R8-80SSE, Package_TO_SOT_SMD:LFPAK88, symbol eswitch:PSMN1R8-80SSE
- added Q31, Q32, Q33, Q34, Q35, Q36, Q37, Q38: FMMT720TA, Package_TO_SOT_SMD:SOT-23, symbol Transistor_BJT:MMBT3906
- added Q6: MMBT3906LT1G, Package_TO_SOT_SMD:SOT-23, symbol Transistor_BJT:MMBT3906
- added R111, R211, R311, R411, R511, R611, R711, R811: 100R, Resistor_SMD:R_0603_1608Metric, symbol Device:R
- added R112, R212: 4.7k 0.1%, Resistor_SMD:R_0603_1608Metric, symbol Device:R
- added R113, R18, R213, R313, R413, R513, R613, R713, R813: 1k 0.1%, Resistor_SMD:R_0603_1608Metric, symbol Device:R
- added R114, R214, R22, R23, R25, R28, R314, R414, R514, R614, R714, R808, R814: 47k, Resistor_SMD:R_0603_1608Metric, symbol Device:R
- added R115, R21, R215, R24, R315, R415, R515, R615, R715, R815: 10k, Resistor_SMD:R_0603_1608Metric, symbol Device:R
- added R116, R117, R216, R217, R316, R317, R416, R417, R516, R517, R616, R617, R716, R717, R816, R817: 10R, Resistor_SMD:R_0603_1608Metric, symbol Device:R
- added R120, R220: 4mR 1% 3W, eswitch:WSLP2512_2m, symbol Device:R
- added R26: 115k 0.1%, Resistor_SMD:R_0603_1608Metric, symbol Device:R
- added R27: 10k 0.1%, Resistor_SMD:R_0603_1608Metric, symbol Device:R
- added R312, R412, R512, R612, R712: 2.2k 0.1%, Resistor_SMD:R_0603_1608Metric, symbol Device:R
- added R320, R420, R520, R620, R720: 8mR 1% 3W, eswitch:WSLP2512_8m, symbol Device:R
- added R812: 7.5k 0.1%, Resistor_SMD:R_0603_1608Metric, symbol Device:R
- added R820: 2mR 1% 3W, eswitch:WSLP2512_2m, symbol Device:R
- added SW10: RESET CH8, Button_Switch_SMD:SW_SPST_PTS645Sx43SMTR92, symbol Switch:SW_Push
- added SW3: RESET CH1, Button_Switch_SMD:SW_SPST_PTS645Sx43SMTR92, symbol Switch:SW_Push
- added SW4: RESET CH2, Button_Switch_SMD:SW_SPST_PTS645Sx43SMTR92, symbol Switch:SW_Push
- added SW5: RESET CH3, Button_Switch_SMD:SW_SPST_PTS645Sx43SMTR92, symbol Switch:SW_Push
- added SW6: RESET CH4, Button_Switch_SMD:SW_SPST_PTS645Sx43SMTR92, symbol Switch:SW_Push
- added SW7: RESET CH5, Button_Switch_SMD:SW_SPST_PTS645Sx43SMTR92, symbol Switch:SW_Push
- added SW8: RESET CH6, Button_Switch_SMD:SW_SPST_PTS645Sx43SMTR92, symbol Switch:SW_Push
- added SW9: RESET CH7, Button_Switch_SMD:SW_SPST_PTS645Sx43SMTR92, symbol Switch:SW_Push
- added TP1: GND, TestPoint:TestPoint_Pad_D1.5mm, symbol Connector:TestPoint
- added TP10: +3V3, TestPoint:TestPoint_Pad_D1.5mm, symbol Connector:TestPoint
- added TP11: MAIN_IMON, TestPoint:TestPoint_Pad_D1.5mm, symbol Connector:TestPoint
- added TP12: MAIN_FLT_N, TestPoint:TestPoint_Pad_D1.5mm, symbol Connector:TestPoint
- added TP13: MAIN_PG_N, TestPoint:TestPoint_Pad_D1.5mm, symbol Connector:TestPoint
- added TP14: BR_ENABLE, TestPoint:TestPoint_Pad_D1.5mm, symbol Connector:TestPoint
- added TP15: ADC_IMON, TestPoint:TestPoint_Pad_D1.5mm, symbol Connector:TestPoint
- added TP16: ADC_BUS, TestPoint:TestPoint_Pad_D1.5mm, symbol Connector:TestPoint
- added TP17: BR_TIMER1, TestPoint:TestPoint_Pad_D1.5mm, symbol Connector:TestPoint
- added TP18: BR_TIMER2, TestPoint:TestPoint_Pad_D1.5mm, symbol Connector:TestPoint
- added TP19: BR_TIMER3, TestPoint:TestPoint_Pad_D1.5mm, symbol Connector:TestPoint
- added TP2: BATT_RAW, TestPoint:TestPoint_Pad_D1.5mm, symbol Connector:TestPoint
- added TP20: BR_TIMER4, TestPoint:TestPoint_Pad_D1.5mm, symbol Connector:TestPoint
- added TP21: BR_TIMER5, TestPoint:TestPoint_Pad_D1.5mm, symbol Connector:TestPoint
- added TP22: BR_TIMER6, TestPoint:TestPoint_Pad_D1.5mm, symbol Connector:TestPoint
- added TP23: BR_TIMER7, TestPoint:TestPoint_Pad_D1.5mm, symbol Connector:TestPoint
- added TP24: BR_TIMER8, TestPoint:TestPoint_Pad_D1.5mm, symbol Connector:TestPoint
- added TP3: BATT_MID, TestPoint:TestPoint_Pad_D1.5mm, symbol Connector:TestPoint
- added TP4: HS_VCC, TestPoint:TestPoint_Pad_D1.5mm, symbol Connector:TestPoint
- added TP5: HS_SENSE, TestPoint:TestPoint_Pad_D1.5mm, symbol Connector:TestPoint
- added TP6: HS_TIMER, TestPoint:TestPoint_Pad_D1.5mm, symbol Connector:TestPoint
- added TP7: HGATE_MAIN, TestPoint:TestPoint_Pad_D1.5mm, symbol Connector:TestPoint
- added TP8: +12V, TestPoint:TestPoint_Pad_D1.5mm, symbol Connector:TestPoint
- added TP9: VIN, TestPoint:TestPoint_Pad_D1.5mm, symbol Connector:TestPoint
- added U21, U22, U23, U24, U25, U26, U27, U28: TPS2492 (CHANNEL LATCH), Package_SO:TSSOP-14_4.4x5mm_P0.65mm, symbol eswitch:TPS2492
- C18: value 10nF 50V C0G 5% -> 12nF 50V C0G 5%; MPN C0805C103J5GACTU -> C0805C123J5GACTU
- C22: renamed from D7; value STPS41L60CG -> 4.7uF 50V; footprint Package_TO_SOT_SMD:TO-263-2 -> Capacitor_SMD:C_1210_3225Metric; symbol eswitch:STPS41L60C -> Device:C; MPN STPS41L60CG-TR -> GRM32ER71H475KA88L; Manufacturer STMicroelectronics -> Murata; Note Both anodes grounded; common cathode/tab on protected bus; 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 -> (none)
- D7: renamed from C104; value 47nF 50V -> STPS41L60CG; footprint Capacitor_SMD:C_0805_2012Metric -> Package_TO_SOT_SMD:TO-263-2; symbol Device:C -> eswitch:STPS41L60C; MPN CL21B473KBCNNNC -> STPS41L60CG-TR; Manufacturer Samsung Electro-Mechanics -> STMicroelectronics; Note VS-to-device-GND EMC capacitor -> Both anodes grounded; common cathode/tab on protected bus; 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
- F1: Note 3 clips per position; CH1 10 A; AUTO: fuse in COM-SW; BYPAS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 -> 3 clips per position; CH1: both AUTO and BYPASS are downstr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
- F2: Note 3 clips per position; CH2 10 A; AUTO: fuse in COM-SW; BYPAS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 -> 3 clips per position; CH2: both AUTO and BYPASS are downstr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
- F3: Note 3 clips per position; CH3 5 A; AUTO: fuse in COM-SW; BYPASS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 -> 3 clips per position; CH3: both AUTO and BYPASS are downstr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
- F4: Note 3 clips per position; CH4 5 A; AUTO: fuse in COM-SW; BYPASS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 -> 3 clips per position; CH4: both AUTO and BYPASS are downstr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
- F5: Note 3 clips per position; CH5 5 A; AUTO: fuse in COM-SW; BYPASS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 -> 3 clips per position; CH5: both AUTO and BYPASS are downstr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
- F6: Note 3 clips per position; CH6 5 A; AUTO: fuse in COM-SW; BYPASS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 -> 3 clips per position; CH6: both AUTO and BYPASS are downstr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
- F7: Note 3 clips per position; CH7 5 A; AUTO: fuse in COM-SW; BYPASS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 -> 3 clips per position; CH7: both AUTO and BYPASS are downstr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
- F8: Note 3 clips per position; CH8 20 A; AUTO: fuse in COM-SW; BYPAS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 -> 3 clips per position; CH8: both AUTO and BYPASS are downstr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
- J12: renamed from J3; value GND IN -> 691218410002; footprint eswitch:ScrewTerminal_Wuerth_74650195_M5 -> eswitch:TerminalBlock_1x02_P7.62mm_Wuerth_2184; symbol Connector:Screw_Terminal_01x01 -> Connector:Screw_Terminal_01x02; MPN 74650195 -> 691218410002; Note M5 ring-lug terminal, 85 A at 20 C component rating; PCB/wi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 -> CH8: pin 1 GND, pin 2 LOAD+; direct-entry screw clamp; 30 A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
- J2: renamed from H4; value M3 -> BATT+ 9.5-16V; footprint MountingHole:MountingHole_3.2mm_M3 -> eswitch:ScrewTerminal_Wuerth_74650195_M5; symbol Mechanical:MountingHole -> Connector:Screw_Terminal_01x01; MPN (none) -> 74650195; Manufacturer (none) -> Wurth Elektronik; Note (none) -> M5 ring-lug terminal, 85 A at 20 C component rating; PCB/wi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; now in the parts list
- J4: footprint Connector_USB:USB_C_Receptacle_GCT_USB4105-xx-A_16P_TopMnt_Horizontal -> eswitch:USB4105_NPTH_0p2
- R16: renamed from R18; value 1k -> 10R; MPN RC0603FR-071KL -> RC0603FR-0710RL
- R17: value 8.25k 1% -> 8.25k 0.1%; MPN RC0603FR-078K25L -> RT0603BRD078K25L
- R20: value 1mR 1% 4W -> 0.5mR 1% 5W; MPN CSS4J-4026R-1L00F -> CSS4J-4026R-L500F; Note Four-terminal shunt; 50 A nominal limit; dedicated sense le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 -> Four-terminal common backup limit; coordinated above one br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
- U14: Note Hardware current/power limiter; timer fault latches until i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 -> Common bus backup current/power limit; branch breakers prov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
- renumbered C204 to C104, C304 to C204, C404 to C304, C504 to C404, C604 to C504, C704 to C604, C804 to C704, R208 to R108, R308 to R208, R408 to R308, R508 to R408, R608 to R508, R708 to R608, R808 to R708
Connections:
- net +12V: now also D7.2 (K_TAB), C113.1, C114.1, C115.1, C116.1, C213.1, C214.1, C215.1, C216.1, C313.1, C314.1, C315.1, C316.1, C413.1, C414.1, C415.1, C416.1, C513.1, C514.1, C515.1, C516.1, C613.1, C614.1, C615.1, C616.1, C713.1, C714.1, C715.1, C716.1, C813.1, C814.1, C815.1, C816.1, R120.1, R220.1, R26.1, R320.1, R420.1, R520.1, R620.1, R720.1, R820.1, TP8.1, U21.14 (VCC), U22.14 (VCC), U23.14 (VCC), U24.14 (VCC), U25.14 (VCC), U26.14 (VCC), U27.14 (VCC), U28.14 (VCC); no longer C22.2 (K_TAB), F1.2 (COM), F2.2 (COM), F3.2 (COM), F4.2 (COM), F5.2 (COM), F6.2 (COM), F7.2 (COM), F8.2 (COM)
- net +3V3: now also D8.2 (K), D9.2 (K), R115.1, R215.1, R24.1, R315.1, R415.1, R515.1, R615.1, R715.1, R815.1, TP10.1
- net BATT_MID: now also TP3.1
- net BATT_RAW: now also J2.1 (Pin_1), TP2.1
- net CAP_USB: now also C22.1
- net GATE_Q3: now also R16.2
- net GND: now also D7.1 (A1), D7.3 (A2), C111.2, C112.2, C113.2, C114.2, C115.2, C116.2, C211.2, C212.2, C213.2, C214.2, C215.2, C216.2, C23.2, C24.2, C25.2, C28.2, C311.2, C312.2, C313.2, C314.2, C315.2, C316.2, C411.2, C412.2, C413.2, C414.2, C415.2, C416.2, C511.2, C512.2, C513.2, C514.2, C515.2, C516.2, C611.2, C612.2, C613.2, C614.2, C615.2, C616.2, C711.2, C712.2, C713.2, C714.2, C715.2, C716.2, C811.2, C812.2, C813.2, C814.2, C815.2, C816.2, D103.1 (A), D111.1 (A1), D111.3 (A2), D112.1 (A), D203.1 (A), D211.1 (A1), D211.3 (A2), D212.1 (A), D303.1 (A), D311.1 (A1), D311.3 (A2), D312.1 (A), D403.1 (A), D411.1 (A1), D411.3 (A2), D412.1 (A), D503.1 (A), D511.1 (A1), D511.3 (A2), D512.1 (A), D603.1 (A), D611.1 (A1), D611.3 (A2), D612.1 (A), D703.1 (A), D711.1 (A1), D711.3 (A2), D712.1 (A), D8.1 (A), D803.1 (A), D811.1 (A1), D811.3 (A2), D812.1 (A), D9.1 (A), J3.1 (Pin_1), R113.2, R18.2, R213.2, R23.2, R27.2, R313.2, R413.2, R513.2, R613.2, R713.2, R813.2, SW10.1, SW3.1, SW4.1, SW5.1, SW6.1, SW7.1, SW8.1, SW9.1, TP1.1, U21.5 (OV), U21.7 (GND), U22.5 (OV), U22.7 (GND), U23.5 (OV), U23.7 (GND), U24.5 (OV), U24.7 (GND), U25.5 (OV), U25.7 (GND), U26.5 (OV), U26.7 (GND), U27.5 (OV), U27.7 (GND), U28.5 (OV), U28.7 (GND); no longer C22.1 (A1), C22.3 (A2), R16.2
- net HGATE_MAIN: now also R16.1, TP7.1
- net HS_PROG: now also R18.1; no longer R16.1
- net HS_REF: now also Q6.2 (E), R22.2
- net HS_SENSE: now also TP5.1
- net HS_TIMER: now also C25.1, C28.1, TP6.1
- net HS_VCC: now also TP4.1
- net IN1: now also U10.8 (IO15); no longer U10.7 (IO7)
- net INR1: now also R108.1
- net INR2: now also R208.1; no longer R108.1
- net INR3: now also R308.1; no longer R208.1
- net INR4: now also R408.1; no longer R308.1
- net INR5: now also R508.1; no longer R408.1
- net INR6: now also R608.1; no longer R508.1
- net INR7: now also R708.1; no longer R608.1
- net INR8: now also R808.1; no longer R708.1
- net LEDK1: now also D103.2 (K)
- net LEDK2: now also D203.2 (K)
- net LEDK3: now also D303.2 (K)
- net LEDK4: now also D403.2 (K)
- net LEDK5: now also D503.2 (K)
- net LEDK6: now also D603.2 (K)
- net LEDK7: now also D703.2 (K)
- net LEDK8: now also D803.2 (K)
- net LOAD8: now also J12.2 (Pin_2)
- net UGND1: now also C104.2, R108.2; no longer D7.2
- net UGND2: now also C204.2, R208.2; no longer C104.2, R108.2
- net UGND3: now also C304.2, R308.2; no longer C204.2, R208.2
- net UGND4: now also C404.2, R408.2; no longer C304.2, R308.2
- net UGND5: now also C504.2, R508.2; no longer C404.2, R408.2
- net UGND6: now also C604.2, R608.2; no longer C504.2, R508.2
- net UGND7: now also C704.2, R708.2; no longer C604.2, R608.2
- net UGND8: now also C804.2, R808.2; no longer C704.2, R708.2
- net VIN: now also C22.2, TP9.1
- net VS1: now also C104.1; no longer D7.1
- net VS2: now also C204.1; no longer C104.1
- net VS3: now also C304.1; no longer C204.1
- net VS4: now also C404.1; no longer C304.1
- net VS5: now also C504.1; no longer C404.1
- net VS6: now also C604.1; no longer C504.1
- net VS7: now also C704.1; no longer C604.1
- net VS8: now also C804.1; no longer C704.1
- net MAIN_IMON: now reaches U14.6 (IMON)
- net MAIN_IMON: now also R25.1, TP11.1
- net MAIN_PG_N: now reaches U14.8 (PG_N)
- net MAIN_PG_N: now also R21.1, TP13.1
- net MAIN_FLT_N: now reaches U14.9 (FLT_N)
- net MAIN_FLT_N: now also U10.35 (IO42), R24.2, TP12.1
- net BR_FLT2: now reaches U10.10 (IO17)
- net BR_FLT2: now also R215.2, U22.9 (FLT_N)
- net BR_FLT3: now reaches U10.11 (IO18)
- net BR_FLT3: now also R315.2, U23.9 (FLT_N)
- net BR_FLT4: now reaches U10.28 (IO35)
- net BR_FLT4: now also R415.2, U24.9 (FLT_N)
- net BR_FLT5: now reaches U10.29 (IO36)
- net BR_FLT5: now also R515.2, U25.9 (FLT_N)
- net BR_FLT6: now reaches U10.30 (IO37)
- net BR_FLT6: now also R615.2, U26.9 (FLT_N)
- net BR_FLT7: now reaches U10.32 (IO39)
- net BR_FLT7: now also R715.2, U27.9 (FLT_N)
- net BR_FLT8: now reaches U10.33 (IO40)
- net BR_FLT8: now also R815.2, U28.9 (FLT_N)
- net ADC_IMON: now reaches U10.5 (IO5)
- net ADC_IMON: now also C23.1, D8.3 (COM), R25.2, TP15.1
- net BR_FLT1: now reaches U10.9 (IO16)
- net BR_FLT1: now also R115.2, U21.9 (FLT_N)
- new net ADC_BUS: C24.1, D9.3 (COM), R28.2, TP16.1, U10.7 (IO7)
- new net BR_EN1: R114.2, SW3.2, U21.1 (UVEN)
- new net BR_EN2: R214.2, SW4.2, U22.1 (UVEN)
- new net BR_EN3: R314.2, SW5.2, U23.1 (UVEN)
- new net BR_EN4: R414.2, SW6.2, U24.1 (UVEN)
- new net BR_EN5: R514.2, SW7.2, U25.1 (UVEN)
- new net BR_EN6: R614.2, SW8.2, U26.1 (UVEN)
- new net BR_EN7: R714.2, SW9.2, U27.1 (UVEN)
- new net BR_EN8: R814.2, SW10.2, U28.1 (UVEN)
- new net BR_ENABLE: Q6.3 (C), R114.1, R214.1, R23.1, R314.1, R414.1, R514.1, R614.1, R714.1, R814.1, TP14.1
- new net BR_ENABLE_BASE: Q6.1 (B), R21.2, R22.1
- new net BR_GATE1: Q31.1 (B), R111.1, U21.12 (GATE)
- new net BR_GATE2: Q32.1 (B), R211.1, U22.12 (GATE)
- new net BR_GATE3: Q33.1 (B), R311.1, U23.12 (GATE)
- new net BR_GATE4: Q34.1 (B), R411.1, U24.12 (GATE)
- new net BR_GATE5: Q35.1 (B), R511.1, U25.12 (GATE)
- new net BR_GATE6: Q36.1 (B), R611.1, U26.12 (GATE)
- new net BR_GATE7: Q37.1 (B), R711.1, U27.12 (GATE)
- new net BR_GATE8: Q38.1 (B), R811.1, U28.12 (GATE)
- new net BR_GS1: Q11.1 (G), Q31.2 (E), R111.2
- new net BR_GS2: Q12.1 (G), Q32.2 (E), R211.2
- new net BR_GS3: Q13.1 (G), Q33.2 (E), R311.2
- new net BR_GS4: Q14.1 (G), Q34.2 (E), R411.2
- new net BR_GS5: Q15.1 (G), Q35.2 (E), R511.2
- new net BR_GS6: Q16.1 (G), Q36.2 (E), R611.2
- new net BR_GS7: Q17.1 (G), Q37.2 (E), R711.2
- new net BR_GS8: Q18.1 (G), Q38.2 (E), R811.2
- new net BR_OUT1: D112.3 (COM), R117.2, U21.11 (OUT)
- new net BR_OUT2: D212.3 (COM), R217.2, U22.11 (OUT)
- new net BR_OUT3: D312.3 (COM), R317.2, U23.11 (OUT)
- new net BR_OUT4: D412.3 (COM), R417.2, U24.11 (OUT)
- new net BR_OUT5: D512.3 (COM), R517.2, U25.11 (OUT)
- new net BR_OUT6: D612.3 (COM), R617.2, U26.11 (OUT)
- new net BR_OUT7: D712.3 (COM), R717.2, U27.11 (OUT)
- new net BR_OUT8: D812.3 (COM), R817.2, U28.11 (OUT)
- new net BR_PROG1: R112.2, R113.1, U21.3 (PROG)
- new net BR_PROG2: R212.2, R213.1, U22.3 (PROG)
- new net BR_PROG3: R312.2, R313.1, U23.3 (PROG)
- new net BR_PROG4: R412.2, R413.1, U24.3 (PROG)
- new net BR_PROG5: R512.2, R513.1, U25.3 (PROG)
- new net BR_PROG6: R612.2, R613.1, U26.3 (PROG)
- new net BR_PROG7: R712.2, R713.1, U27.3 (PROG)
- new net BR_PROG8: R812.2, R813.1, U28.3 (PROG)
- new net BR_PULL1: Q31.3 (C), R116.1
- new net BR_PULL2: Q32.3 (C), R216.1
- new net BR_PULL3: Q33.3 (C), R316.1
- new net BR_PULL4: Q34.3 (C), R416.1
- new net BR_PULL5: Q35.3 (C), R516.1
- new net BR_PULL6: Q36.3 (C), R616.1
- new net BR_PULL7: Q37.3 (C), R716.1
- new net BR_PULL8: Q38.3 (C), R816.1
- new net BR_REF1: R112.1, U21.2 (VREF)
- new net BR_REF2: R212.1, U22.2 (VREF)
- new net BR_REF3: R312.1, U23.2 (VREF)
- new net BR_REF4: R412.1, U24.2 (VREF)
- new net BR_REF5: R512.1, U25.2 (VREF)
- new net BR_REF6: R612.1, U26.2 (VREF)
- new net BR_REF7: R712.1, U27.2 (VREF)
- new net BR_REF8: R812.1, U28.2 (VREF)
- new net BR_SENSE1: Q11.5 (D_MB), R120.2, U21.13 (SENSE)
- new net BR_SENSE2: Q12.5 (D_MB), R220.2, U22.13 (SENSE)
- new net BR_SENSE3: Q13.5 (D_MB), R320.2, U23.13 (SENSE)
- new net BR_SENSE4: Q14.5 (D_MB), R420.2, U24.13 (SENSE)
- new net BR_SENSE5: Q15.5 (D_MB), R520.2, U25.13 (SENSE)
- new net BR_SENSE6: Q16.5 (D_MB), R620.2, U26.13 (SENSE)
- new net BR_SENSE7: Q17.5 (D_MB), R720.2, U27.13 (SENSE)
- new net BR_SENSE8: Q18.5 (D_MB), R820.2, U28.13 (SENSE)
- new net BR_TIMER1: C111.1, C112.1, TP17.1, U21.4 (TIMER)
- new net BR_TIMER2: C211.1, C212.1, TP18.1, U22.4 (TIMER)
- new net BR_TIMER3: C311.1, C312.1, TP19.1, U23.4 (TIMER)
- new net BR_TIMER4: C411.1, C412.1, TP20.1, U24.4 (TIMER)
- new net BR_TIMER5: C511.1, C512.1, TP21.1, U25.4 (TIMER)
- new net BR_TIMER6: C611.1, C612.1, TP22.1, U26.4 (TIMER)
- new net BR_TIMER7: C711.1, C712.1, TP23.1, U27.4 (TIMER)
- new net BR_TIMER8: C811.1, C812.1, TP24.1, U28.4 (TIMER)
- new net BUS_DIV: R26.2, R27.1, R28.1
- new net CHFEED1: D111.2 (K_TAB), F1.2 (COM), Q11.2 (S), Q11.3 (S), Q11.4 (S), R116.2, R117.1
- new net CHFEED2: D211.2 (K_TAB), F2.2 (COM), Q12.2 (S), Q12.3 (S), Q12.4 (S), R216.2, R217.1
- new net CHFEED3: D311.2 (K_TAB), F3.2 (COM), Q13.2 (S), Q13.3 (S), Q13.4 (S), R316.2, R317.1
- new net CHFEED4: D411.2 (K_TAB), F4.2 (COM), Q14.2 (S), Q14.3 (S), Q14.4 (S), R416.2, R417.1
- new net CHFEED5: D511.2 (K_TAB), F5.2 (COM), Q15.2 (S), Q15.3 (S), Q15.4 (S), R516.2, R517.1
- new net CHFEED6: D611.2 (K_TAB), F6.2 (COM), Q16.2 (S), Q16.3 (S), Q16.4 (S), R616.2, R617.1
- new net CHFEED7: D711.2 (K_TAB), F7.2 (COM), Q17.2 (S), Q17.3 (S), Q17.4 (S), R716.2, R717.1
- new net CHFEED8: D811.2 (K_TAB), F8.2 (COM), Q18.2 (S), Q18.3 (S), Q18.4 (S), R816.2, R817.1
- no-connect marks 23 -> 41
Other:
- note added: "MCU: IS1-8 -> ADC1 IO1,3,4,2,6,10,8,9; IN1 -> IO15; IMON -> IO5; BUS -> IO7; see pin map"
- note removed: "MCU: ESP32-S3-WROOM-1 (IS1-8 -> ADC1 IO1,3,4,2,6,10,8,9; IN1-8 -> IO7,11,12,13,14,21,47,48; DEN -> IO38; STAT LED -> IO41)"
- title: eswitch - 8ch PROFET load switch -> eswitch - 8 independent latching channels
- moved on the sheet: C104, C204, C304, C404, C504, C604, C704, R108, R16, R208, R308, R408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
