File: redesign/eswitch-simple.kicad_sch (KiCad schematic)
At the start: 210 parts, among them J11 CH1 OUTPUT, J12 CH2 OUTPUT, J13 CH3 OUTPUT, J14 CH4 OUTPUT, J15 CH5 OUTPUT, J16 CH6 OUTPUT, J17 CH7 OUTPUT, J18 CH8 OUTPUT, J2 BATT_RAW, J3 GND, J4 USB-C, J5 UART, Q5 BSC016N06NS, SW1 RESET, SW2 BOOT, U1 BTS7004-1EPP, U10 ESP32-S3-WROOM-1-N8, U11 SRV05-4HTG-D, U13 LM74800-Q1, U14 TLA431AIDBZR, U2 BTS7004-1EPP, U3 BTS7008-1EPR, U4 BTS7008-1EPR, U5 BTS7008-1EPR, U6 BTS7008-1EPR, U7 BTS7008-1EPR, U8 BTS7002-1EPP, U9 TPSM63603V3

Commit message: Rework power copper and package expanded prototype for fabrication
Connections:
- net GND: now also J11.2 (Pin_2), J12.2 (Pin_2), J13.2 (Pin_2), J14.2 (Pin_2), J15.2 (Pin_2), J16.2 (Pin_2), J17.2 (Pin_2), J18.2 (Pin_2); no longer J11.1 (Pin_1), J12.1 (Pin_1), J13.1 (Pin_1), J14.1 (Pin_1), J15.1 (Pin_1), J16.1 (Pin_1), J17.1 (Pin_1), J18.1 (Pin_1)
- net LOAD1: now also J11.1 (Pin_1); no longer J11.2 (Pin_2)
- net LOAD2: now also J12.1 (Pin_1); no longer J12.2 (Pin_2)
- net LOAD3: now also J13.1 (Pin_1); no longer J13.2 (Pin_2)
- net LOAD4: now also J14.1 (Pin_1); no longer J14.2 (Pin_2)
- net LOAD5: now also J15.1 (Pin_1); no longer J15.2 (Pin_2)
- net LOAD6: now also J16.1 (Pin_1); no longer J16.2 (Pin_2)
- net LOAD7: now also J17.1 (Pin_1); no longer J17.2 (Pin_2)
- net LOAD8: now also J18.1 (Pin_1); no longer J18.2 (Pin_2)
Other:
- note added: "ESWITCH SIMPLE — PROTOTYPE / BENCH QUALIFICATION REQUIRED"
- note added: "OUTPUTS: pin 1 LOAD+, pin 2 GND; direct-entry screw terminals"
- note removed: "ESWITCH SIMPLE — ENGINEERING DRAFT / NOT FOR FABRICATION"
- note removed: "OUTPUTS: pin 1 GND, pin 2 LOAD+; direct-entry screw terminals"
Changed lines of the file:
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@@
 	(title_block
 		(title "eswitch simple — passive fuse bypass")
-		(date "2026-10-25")
-		(rev "DRAFT-1")
+		(date "2026-10-26")
+		(rev "DRAFT-PWR2")
 	)
 	(symbol
@@
 		)
 	)
-	(label "GND"
+	(label "LOAD1"
 		(at 332.74 269.24 180)
 		(effects
@@
 		)
 	)
-	(label "LOAD1"
+	(label "GND"
 		(at 332.74 271.78 180)
 		(effects
@@
 		)
 	)
-	(label "GND"
+	(label "LOAD2"
 		(at 363.22 269.24 180)
 		(effects
@@
 		)
 	)
-	(label "LOAD2"
+	(label "GND"
 		(at 363.22 271.78 180)
 		(effects
@@
 		)
 	)
-	(label "GND"
+	(label "LOAD3"
 		(at 393.7 269.24 180)
 		(effects
@@
 		)
 	)
-	(label "LOAD3"
+	(label "GND"
 		(at 393.7 271.78 180)
 		(effects
@@
 		)
 	)
-	(label "GND"
+	(label "LOAD4"
 		(at 424.18 269.24 180)
 		(effects
@@
 		)
 	)
-	(label "LOAD4"
+	(label "GND"
 		(at 424.18 271.78 180)
 		(effects
@@
 		)
 	)
-	(label "GND"
+	(label "LOAD5"
 		(at 332.74 294.64 180)
 		(effects
@@
 		)
 	)
-	(label "LOAD5"
+	(label "GND"
 		(at 332.74 297.18 180)
 		(effects
@@
 		)
 	)
-	(label "GND"
+	(label "LOAD6"
 		(at 363.22 294.64 180)
 		(effects
@@
 		)
 	)
-	(label "LOAD6"
+	(label "GND"
 		(at 363.22 297.18 180)
 		(effects
@@
 		)
 	)
-	(label "GND"
+	(label "LOAD7"
 		(at 393.7 294.64 180)
 		(effects
@@
 		)
 	)
-	(label "LOAD7"
+	(label "GND"
 		(at 393.7 297.18 180)
 		(effects
@@
 		)
 	)
-	(label "GND"
+	(label "LOAD8"
 		(at 424.18 294.64 180)
 		(effects
@@
 		)
 	)
-	(label "LOAD8"
+	(label "GND"
 		(at 424.18 297.18 180)
 		(effects
@@
 		)
 	)
-	(text "ESWITCH SIMPLE — ENGINEERING DRAFT / NOT FOR FABRICATION"
+	(text "ESWITCH SIMPLE — PROTOTYPE / BENCH QUALIFICATION REQUIRED"
 		(exclude_from_sim no)
 		(at 12.7 17.78 0)
@@
 		)
 	)
-	(text "OUTPUTS: pin 1 GND, pin 2 LOAD+; direct-entry screw terminals"
+	(text "OUTPUTS: pin 1 LOAD+, pin 2 GND; direct-entry screw terminals"
 		(exclude_from_sim no)
 		(at 330.2 246.38 0)

Commit message: Release PROTO-PWR3 shared AUTO protection and passive bypass prototype
Parts:
- removed C2: 4.7uF 50V, Capacitor_SMD:C_1210_3225Metric, symbol Device:C
- removed C3: 100nF 50V, Capacitor_SMD:C_0805_2012Metric, symbol Device:C
- removed C303, C403, C503, C603: 10nF 50V, Capacitor_SMD:C_0805_2012Metric, symbol Device:C
- removed C504, C604: 47nF 50V, Capacitor_SMD:C_0805_2012Metric, symbol Device:C
- removed D103, D201, D203, D301, D303, D401, D403, D501, D503, D601, D603, D701, D703, D803: BAT54S, Package_TO_SOT_SMD:SOT-23, symbol Diode:BAT54S
- removed D204, D304, D404, D504, D604, D704, D804: SMCJ16A, Diode_SMD:D_SMC, symbol Device:D_TVS
- removed D5: BLUE, LED_SMD:LED_0603_1608Metric, symbol Device:LED
- removed H7: M3 mounting / 10mm standoff, MountingHole:MountingHole_3.2mm_M3, symbol Mechanical:MountingHole
- removed J16: CH6 OUTPUT, eswitch:TerminalBlock_1x02_P7.62mm_Wuerth_2184, symbol Connector:Screw_Terminal_01x02
- removed J17: CH7 OUTPUT, eswitch:TerminalBlock_1x02_P7.62mm_Wuerth_2184, symbol Connector:Screw_Terminal_01x02
- removed J18: CH8 OUTPUT, eswitch:TerminalBlock_1x02_P7.62mm_Wuerth_2184, symbol Connector:Screw_Terminal_01x02
- removed J2: BATT_RAW, eswitch:ScrewTerminal_Wuerth_74650195_M5, symbol Connector:Screw_Terminal_01x01
- removed J5: UART, Connector_PinHeader_2.54mm:PinHeader_1x04_P2.54mm_Vertical, symbol Connector_Generic:Conn_01x04
- removed R309, R408, R409, R508, R509, R608, R609, R708, R709, R809: 47k, Resistor_SMD:R_0603_1608Metric, symbol Device:R
- removed R403, R503: 47R, Resistor_SMD:R_0805_2012Metric, symbol Device:R
- removed R704: 3.3k, Resistor_SMD:R_0603_1608Metric, symbol Device:R
- removed R805: 4.7k, Resistor_SMD:R_0603_1608Metric, symbol Device:R
- removed U9: TPSM63603V3, eswitch:TI_RDH0030A_TPSM63603, symbol eswitch:TPSM63603V3
- added C10, C201, C24, C301, C401, C501, C601, C701, C801: 100nF 50V, Capacitor_SMD:C_0805_2012Metric, symbol Device:C
- added C25: 100nF 250V, Capacitor_SMD:C_1210_3225Metric, symbol Device:C
- added C26, C28: 1uF 100V, Capacitor_SMD:C_1210_3225Metric, symbol Device:C
- added C27: 1uF 50V, Capacitor_SMD:C_0805_2012Metric, symbol Device:C
- added C29: 4.7uF 50V, Capacitor_SMD:C_1210_3225Metric, symbol Device:C
- added C302, C402, C502, C602, C702, C802: 10nF 50V, Capacitor_SMD:C_0805_2012Metric, symbol Device:C
- added C9: 10uF 10V, Capacitor_SMD:C_0805_2012Metric, symbol Device:C
- added D10: SMCJ16A LOCAL TRANSIENT, Diode_SMD:D_SMC, symbol Device:D_TVS
- added D6: SMBJ150A, Diode_SMD:D_SMB, symbol Device:D_TVS
- added D7: SMBJ33CA, Diode_SMD:D_SMB, symbol Device:D_TVS
- added D8: 51V 2%, Diode_SMD:D_SMA, symbol Device:D_Zener
- added D9: 82V, Diode_SMD:D_SMA, symbol Device:D_Zener
- added F10: 40A AUTO/LOGIC ISOLATION, eswitch:Fuse_Mersen_14x51_MR14_Wuerth_M5, symbol Device:Fuse
- added H4: M3 mounting / 10mm standoff, MountingHole:MountingHole_3.2mm_M3, symbol Mechanical:MountingHole
- added J11: CH1 OUTPUT, eswitch:TerminalBlock_1x02_P7.62mm_Wuerth_2184, symbol Connector:Screw_Terminal_01x02
- added J13: CH3 OUTPUT, eswitch:TerminalBlock_1x02_P7.62mm_Wuerth_2184, symbol Connector:Screw_Terminal_01x02
- added Q10, Q11: BSC016N06NS 60V, Package_SON:Infineon_PG-TDSON-8_6.15x5.15mm, symbol eswitch:BSC016N06NS
- added Q6, Q7, Q8, Q9: IPT067N20NM6 200V, Package_TO_SOT_SMD:Infineon_PG-HSOF-8-1, symbol Transistor_FET:IPT012N08N5
- added R10: 22R, Resistor_SMD:R_0603_1608Metric, symbol Device:R
- added R14: 2.2k, Resistor_SMD:R_0603_1608Metric, symbol Device:R
- added R15, R406, R506, R606, R706: 47k, Resistor_SMD:R_0603_1608Metric, symbol Device:R
- added R20, R21, R23, R24, R25: 10R, Resistor_SMD:R_0805_2012Metric, symbol Device:R
- added R201, R301, R302, R401, R402, R502, R601, R701: 4.7k, Resistor_SMD:R_0603_1608Metric, symbol Device:R
- added R26: 4.7k 2W, Resistor_THT:R_Axial_DIN0411_L9.9mm_D3.6mm_P15.24mm_Horizontal, symbol Device:R
- added R27, R28: 49.9k 0.1%, Resistor_SMD:R_0805_2012Metric, symbol Device:R
- added R29: 7.87k 0.1%, Resistor_SMD:R_0805_2012Metric, symbol Device:R
- added R404, R504: 3.3k, Resistor_SMD:R_0603_1608Metric, symbol Device:R
- added R507, R607: 10k, Resistor_SMD:R_0603_1608Metric, symbol Device:R
- added R7, R8: 5.1k, Resistor_SMD:R_0603_1608Metric, symbol Device:R
- added U15: LM74800-Q1 AUTO CUTOFF, Package_SON:WSON-12-1EP_3x3mm_P0.5mm_EP1.5x2.5mm, symbol eswitch:LM74800
- added U5, U6, U7: BTS7008-1EPR, Package_SO:Infineon_PG-TSDSO-14-22, symbol eswitch:BTS7008-1EPR
- added U8: BTS7002-1EPP, Package_SO:Infineon_PG-TSDSO-14-22, symbol eswitch:BTS7002-1EPP
- C2: renamed from R7; value 5.1k -> 4.7uF 50V; footprint Resistor_SMD:R_0603_1608Metric -> Capacitor_SMD:C_1210_3225Metric; symbol Device:R -> Device:C; MPN ERJ-3EKF5101V -> GRM32ER71H475KA88L
- C202: renamed from C201; value 100nF 50V -> 10nF 50V; MPN CL21B104KBCNNNC -> CL21B103KBANNNC
- C203: renamed from R203; value 47R -> 10nF 50V; footprint Resistor_SMD:R_0805_2012Metric -> Capacitor_SMD:C_0805_2012Metric; symbol Device:R -> Device:C; MPN RC0805FR-0747RL -> CL21B103KBANNNC
- C204: renamed from D202; value GREEN -> 47nF 50V; footprint LED_SMD:LED_0603_1608Metric -> Capacitor_SMD:C_0805_2012Metric; symbol Device:LED -> Device:C; MPN 150060GS75000 -> CL21B473KBCNNNC
- C3: renamed from R8; value 5.1k -> 100nF 50V; footprint Resistor_SMD:R_0603_1608Metric -> Capacitor_SMD:C_0805_2012Metric; symbol Device:R -> Device:C; MPN ERJ-3EKF5101V -> CL21B104KBCNNNC
- C303: renamed from R305; value 4.7k -> 10nF 50V; footprint Resistor_SMD:R_0603_1608Metric -> Capacitor_SMD:C_0805_2012Metric; symbol Device:R -> Device:C; MPN RC0603FR-074K7L -> CL21B103KBANNNC
- C304: renamed from R307; value 10k -> 47nF 50V; footprint Resistor_SMD:R_0603_1608Metric -> Capacitor_SMD:C_0805_2012Metric; symbol Device:R -> Device:C; MPN RC0603FR-0710KL -> CL21B473KBCNNNC
- C403: renamed from R404; value 3.3k -> 10nF 50V; footprint Resistor_SMD:R_0603_1608Metric -> Capacitor_SMD:C_0805_2012Metric; symbol Device:R -> Device:C; MPN RC0603FR-073K3L -> CL21B103KBANNNC
- C404: renamed from R406; value 47k -> 47nF 50V; footprint Resistor_SMD:R_0603_1608Metric -> Capacitor_SMD:C_0805_2012Metric; symbol Device:R -> Device:C; MPN RC0603FR-0747KL -> CL21B473KBCNNNC
- C503: renamed from R502; value 4.7k -> 10nF 50V; footprint Resistor_SMD:R_0603_1608Metric -> Capacitor_SMD:C_0805_2012Metric; symbol Device:R -> Device:C; MPN RC0603FR-074K7L -> CL21B103KBANNNC
- C504: renamed from C502; value 10nF 50V -> 47nF 50V; MPN CL21B103KBANNNC -> CL21B473KBCNNNC
- C603: renamed from R601; value 4.7k -> 10nF 50V; footprint Resistor_SMD:R_0603_1608Metric -> Capacitor_SMD:C_0805_2012Metric; symbol Device:R -> Device:C; MPN RC0603FR-074K7L -> CL21B103KBANNNC
- C604: renamed from C601; value 100nF 50V -> 47nF 50V; MPN CL21B104KBCNNNC -> CL21B473KBCNNNC
- D103: renamed from D104; value SMCJ16A -> BAT54S; footprint Diode_SMD:D_SMC -> Package_TO_SOT_SMD:SOT-23; symbol Device:D_TVS -> Diode:BAT54S; MPN SMCJ16A -> BAT54S-QR; Note Candidate local clamp; transient energy and inductive turn-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 -> (none)
- D201: renamed from C203; value 10nF 50V -> BAT54S; footprint Capacitor_SMD:C_0805_2012Metric -> Package_TO_SOT_SMD:SOT-23; symbol Device:C -> Diode:BAT54S; MPN CL21B103KBANNNC -> BAT54S-QR
- D202: renamed from R207; value 10k -> GREEN; footprint Resistor_SMD:R_0603_1608Metric -> LED_SMD:LED_0603_1608Metric; symbol Device:R -> Device:LED; MPN RC0603FR-0710KL -> 150060GS75000
- D203: renamed from R209; value 47k -> BAT54S; footprint Resistor_SMD:R_0603_1608Metric -> Package_TO_SOT_SMD:SOT-23; symbol Device:R -> Diode:BAT54S; MPN RC0603FR-0747KL -> BAT54S-QR
- D301: renamed from R303; value 47R -> BAT54S; footprint Resistor_SMD:R_0805_2012Metric -> Package_TO_SOT_SMD:SOT-23; symbol Device:R -> Diode:BAT54S; MPN RC0805FR-0747RL -> BAT54S-QR
- D302: renamed from R306; value 47k -> GREEN; footprint Resistor_SMD:R_0603_1608Metric -> LED_SMD:LED_0603_1608Metric; symbol Device:R -> Device:LED; MPN RC0603FR-0747KL -> 150060GS75000
- D303: renamed from R308; value 47k -> BAT54S; footprint Resistor_SMD:R_0603_1608Metric -> Package_TO_SOT_SMD:SOT-23; symbol Device:R -> Diode:BAT54S; MPN RC0603FR-0747KL -> BAT54S-QR
- D401: renamed from R405; value 4.7k -> BAT54S; footprint Resistor_SMD:R_0603_1608Metric -> Package_TO_SOT_SMD:SOT-23; symbol Device:R -> Diode:BAT54S; MPN RC0603FR-074K7L -> BAT54S-QR
- D402: renamed from C402; value 10nF 50V -> GREEN; footprint Capacitor_SMD:C_0805_2012Metric -> LED_SMD:LED_0603_1608Metric; symbol Device:C -> Device:LED; MPN CL21B103KBANNNC -> 150060GS75000
- D403: renamed from C404; value 47nF 50V -> BAT54S; footprint Capacitor_SMD:C_0805_2012Metric -> Package_TO_SOT_SMD:SOT-23; symbol Device:C -> Diode:BAT54S; MPN CL21B473KBCNNNC -> BAT54S-QR
- D5: renamed from C9; value 10uF 10V -> BLUE; footprint Capacitor_SMD:C_0805_2012Metric -> LED_SMD:LED_0603_1608Metric; symbol Device:C -> Device:LED; MPN CC0805KKX5R6BB106 -> 150060BS75000
- D501: renamed from R504; value 3.3k -> BAT54S; footprint Resistor_SMD:R_0603_1608Metric -> Package_TO_SOT_SMD:SOT-23; symbol Device:R -> Diode:BAT54S; MPN RC0603FR-073K3L -> BAT54S-QR
- D502: renamed from C501; value 100nF 50V -> GREEN; footprint Capacitor_SMD:C_0805_2012Metric -> LED_SMD:LED_0603_1608Metric; symbol Device:C -> Device:LED; MPN CL21B104KBCNNNC -> 150060GS75000
- D503: renamed from D502; value GREEN -> BAT54S; footprint LED_SMD:LED_0603_1608Metric -> Package_TO_SOT_SMD:SOT-23; symbol Device:LED -> Diode:BAT54S; MPN 150060GS75000 -> BAT54S-QR
- D601: renamed from R602; value 4.7k -> BAT54S; footprint Resistor_SMD:R_0603_1608Metric -> Package_TO_SOT_SMD:SOT-23; symbol Device:R -> Diode:BAT54S; MPN RC0603FR-074K7L -> BAT54S-QR
- D603: renamed from R607; value 10k -> BAT54S; footprint Resistor_SMD:R_0603_1608Metric -> Package_TO_SOT_SMD:SOT-23; symbol Device:R -> Diode:BAT54S; MPN RC0603FR-0710KL -> BAT54S-QR
- D701: renamed from R701; value 4.7k -> BAT54S; footprint Resistor_SMD:R_0603_1608Metric -> Package_TO_SOT_SMD:SOT-23; symbol Device:R -> Diode:BAT54S; MPN RC0603FR-074K7L -> BAT54S-QR
- D703: renamed from R706; value 47k -> BAT54S; footprint Resistor_SMD:R_0603_1608Metric -> Package_TO_SOT_SMD:SOT-23; symbol Device:R -> Diode:BAT54S; MPN RC0603FR-0747KL -> BAT54S-QR
- D803: renamed from C802; value 10nF 50V -> BAT54S; footprint Capacitor_SMD:C_0805_2012Metric -> Package_TO_SOT_SMD:SOT-23; symbol Device:C -> Diode:BAT54S; MPN CL21B103KBANNNC -> BAT54S-QR
- F1, F2, F3, F4, F5, F6, F7, F8: Note ONE fuse: AUTO COM-SW; BYPASS COM-LOAD; remove for OFF. Cha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 -> ONE fuse: AUTO OUT-LOAD; BYPASS RAW-LOAD; remove for OFF. C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
- H7: renamed from J13; value CH3 OUTPUT -> M3 mounting / 10mm standoff; footprint eswitch:TerminalBlock_1x02_P7.62mm_Wuerth_2184 -> MountingHole:MountingHole_3.2mm_M3; symbol Connector:Screw_Terminal_01x02 -> Mechanical:MountingHole; MPN 691218410002 -> R30-1001002; Note (none) -> BOM item is the M3 standoff; hole itself is unplated; now left out of the parts list
- J16: renamed from R14; value 2.2k -> CH6 OUTPUT; footprint Resistor_SMD:R_0603_1608Metric -> eswitch:TerminalBlock_1x02_P7.62mm_Wuerth_2184; symbol Device:R -> Connector:Screw_Terminal_01x02; MPN RC0603FR-072K2L -> 691218410002
- J17: renamed from R15; value 47k -> CH7 OUTPUT; footprint Resistor_SMD:R_0603_1608Metric -> eswitch:TerminalBlock_1x02_P7.62mm_Wuerth_2184; symbol Device:R -> Connector:Screw_Terminal_01x02; MPN RC0603FR-0747KL -> 691218410002
- J18: renamed from C24; value 100nF 50V -> CH8 OUTPUT; footprint Capacitor_SMD:C_0805_2012Metric -> eswitch:TerminalBlock_1x02_P7.62mm_Wuerth_2184; symbol Device:C -> Connector:Screw_Terminal_01x02; MPN CL21B104KBCNNNC -> 691218410002
- J2: renamed from J11; value CH1 OUTPUT -> BATT_RAW; footprint eswitch:TerminalBlock_1x02_P7.62mm_Wuerth_2184 -> eswitch:ScrewTerminal_Wuerth_74650195_M5; symbol Connector:Screw_Terminal_01x02 -> Connector:Screw_Terminal_01x01; MPN 691218410002 -> 74650195
- J5: renamed from C10; value 100nF 50V -> UART; footprint Capacitor_SMD:C_0805_2012Metric -> Connector_PinHeader_2.54mm:PinHeader_1x04_P2.54mm_Vertical; symbol Device:C -> Connector_Generic:Conn_01x04; MPN CL21B104KBCNNNC -> 61300411121
- R104: MPN RC0603FR-072K2L -> ERJ-PA3F2201V; Note (none) -> High-power 0603 sense resistor; retain value, use ERJ-PA3 p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
- R203: renamed from R205; value 4.7k -> 47R; footprint Resistor_SMD:R_0603_1608Metric -> Resistor_SMD:R_0805_2012Metric; MPN RC0603FR-074K7L -> RC0805FR-0747RL
- R204: renamed from R202; value 4.7k -> 2.2k; MPN RC0603FR-074K7L -> ERJ-PA3F2201V; Note (none) -> High-power 0603 sense resistor; retain value, use ERJ-PA3 p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
- R205: renamed from R204; value 2.2k -> 4.7k; MPN RC0603FR-072K2L -> RC0603FR-074K7L
- R206: renamed from C202; value 10nF 50V -> 47k; footprint Capacitor_SMD:C_0805_2012Metric -> Resistor_SMD:R_0603_1608Metric; symbol Device:C -> Device:R; MPN CL21B103KBANNNC -> RC0603FR-0747KL
- R207: renamed from R206; value 47k -> 10k; MPN RC0603FR-0747KL -> RC0603FR-0710KL
- R208: renamed from C204; value 47nF 50V -> 47k; footprint Capacitor_SMD:C_0805_2012Metric -> Resistor_SMD:R_0603_1608Metric; symbol Device:C -> Device:R; MPN CL21B473KBCNNNC -> RC0603FR-0747KL
- R22: renamed from H4; value M3 mounting / 10mm standoff -> 10R; footprint MountingHole:MountingHole_3.2mm_M3 -> Resistor_SMD:R_0805_2012Metric; symbol Mechanical:MountingHole -> Device:R; MPN R30-1001002 -> RC0805FR-0710RL; Note BOM item is the M3 standoff; hole itself is unplated -> (none); now in the parts list
- R303: renamed from R304; value 3.3k -> 47R; footprint Resistor_SMD:R_0603_1608Metric -> Resistor_SMD:R_0805_2012Metric; MPN RC0603FR-073K3L -> RC0805FR-0747RL
- R304: renamed from R301; value 4.7k -> 3.3k; MPN RC0603FR-074K7L -> ERJ-PA3F3301V; Note (none) -> High-power 0603 sense resistor; retain value, use ERJ-PA3 p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
- R306: renamed from C301; value 100nF 50V -> 47k; footprint Capacitor_SMD:C_0805_2012Metric -> Resistor_SMD:R_0603_1608Metric; symbol Device:C -> Device:R; MPN CL21B104KBCNNNC -> RC0603FR-0747KL
- R307: renamed from C302; value 10nF 50V -> 10k; footprint Capacitor_SMD:C_0805_2012Metric -> Resistor_SMD:R_0603_1608Metric; symbol Device:C -> Device:R; MPN CL21B103KBANNNC -> RC0603FR-0710KL
- R308: renamed from D302; value GREEN -> 47k; footprint LED_SMD:LED_0603_1608Metric -> Resistor_SMD:R_0603_1608Metric; symbol Device:LED -> Device:R; MPN 150060GS75000 -> RC0603FR-0747KL
- R309: renamed from C304; value 47nF 50V -> 47k; footprint Capacitor_SMD:C_0805_2012Metric -> Resistor_SMD:R_0603_1608Metric; symbol Device:C -> Device:R; MPN CL21B473KBCNNNC -> RC0603FR-0747KL
- R403: renamed from R402; value 4.7k -> 47R; footprint Resistor_SMD:R_0603_1608Metric -> Resistor_SMD:R_0805_2012Metric; MPN RC0603FR-074K7L -> RC0805FR-0747RL
- R407: renamed from C401; value 100nF 50V -> 10k; footprint Capacitor_SMD:C_0805_2012Metric -> Resistor_SMD:R_0603_1608Metric; symbol Device:C -> Device:R; MPN CL21B104KBCNNNC -> RC0603FR-0710KL
- R408: renamed from R407; value 10k -> 47k; MPN RC0603FR-0710KL -> RC0603FR-0747KL
- R409: renamed from D402; value GREEN -> 47k; footprint LED_SMD:LED_0603_1608Metric -> Resistor_SMD:R_0603_1608Metric; symbol Device:LED -> Device:R; MPN 150060GS75000 -> RC0603FR-0747KL
- R501: renamed from U5; value BTS7008-1EPR -> 4.7k; footprint Package_SO:Infineon_PG-TSDSO-14-22 -> Resistor_SMD:R_0603_1608Metric; symbol eswitch:BTS7008-1EPR -> Device:R; MPN BTS70081EPRXUMA1 -> RC0603FR-074K7L
- R503: renamed from R501; value 4.7k -> 47R; footprint Resistor_SMD:R_0603_1608Metric -> Resistor_SMD:R_0805_2012Metric; MPN RC0603FR-074K7L -> RC0805FR-0747RL
- R509: renamed from R507; value 10k -> 47k; MPN RC0603FR-0710KL -> RC0603FR-0747KL
- R602: renamed from U6; value BTS7008-1EPR -> 4.7k; footprint Package_SO:Infineon_PG-TSDSO-14-22 -> Resistor_SMD:R_0603_1608Metric; symbol eswitch:BTS7008-1EPR -> Device:R; MPN BTS70081EPRXUMA1 -> RC0603FR-074K7L
- R604: MPN RC0603FR-073K3L -> ERJ-PA3F3301V; Note (none) -> High-power 0603 sense resistor; retain value, use ERJ-PA3 p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
- R608: renamed from C602; value 10nF 50V -> 47k; footprint Capacitor_SMD:C_0805_2012Metric -> Resistor_SMD:R_0603_1608Metric; symbol Device:C -> Device:R; MPN CL21B103KBANNNC -> RC0603FR-0747KL
- R704: renamed from U7; value BTS7008-1EPR -> 3.3k; footprint Package_SO:Infineon_PG-TSDSO-14-22 -> Resistor_SMD:R_0603_1608Metric; symbol eswitch:BTS7008-1EPR -> Device:R; MPN BTS70081EPRXUMA1 -> ERJ-PA3F3301V; Note (none) -> High-power 0603 sense resistor; retain value, use ERJ-PA3 p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
- R708: renamed from C701; value 100nF 50V -> 47k; footprint Capacitor_SMD:C_0805_2012Metric -> Resistor_SMD:R_0603_1608Metric; symbol Device:C -> Device:R; MPN CL21B104KBCNNNC -> RC0603FR-0747KL
- R709: renamed from C702; value 10nF 50V -> 47k; footprint Capacitor_SMD:C_0805_2012Metric -> Resistor_SMD:R_0603_1608Metric; symbol Device:C -> Device:R; MPN CL21B103KBANNNC -> RC0603FR-0747KL
- R804: MPN RC0603FR-071K2L -> ERJ-PA3F1201V; Note (none) -> High-power 0603 sense resistor; retain value, use ERJ-PA3 p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
- R805: renamed from U8; value BTS7002-1EPP -> 4.7k; footprint Package_SO:Infineon_PG-TSDSO-14-22 -> Resistor_SMD:R_0603_1608Metric; symbol eswitch:BTS7002-1EPP -> Device:R; MPN BTS70021EPPXUMA1 -> RC0603FR-074K7L
- R809: renamed from C801; value 100nF 50V -> 47k; footprint Capacitor_SMD:C_0805_2012Metric -> Resistor_SMD:R_0603_1608Metric; symbol Device:C -> Device:R; MPN CL21B104KBCNNNC -> RC0603FR-0747KL
- U9: renamed from R10; value 22R -> TPSM63603V3; footprint Resistor_SMD:R_0603_1608Metric -> eswitch:TI_RDH0030A_TPSM63603; symbol Device:R -> eswitch:TPSM63603V3; MPN ERJ-3EKF22R0V -> TPSM63603V3RDHR
- renumbered R201 to R202, R208 to R209, R302 to R305, R401 to R405, R506 to R508, R606 to R609
Connections:
- net +3V3: now also J5.2 (Pin_2), U9.10 (VOUT), U9.12 (VOUT), U9.13 (VOUT), U9.14 (VOUT), U9.15 (VOUT), U9.22 (VLDOIN), U9.25 (FB), U9.30 (VOUT), U9.7 (VOUT), U9.8 (VOUT), U9.9 (VOUT), C10.1, C9.1, R14.1; no longer D5.1, J16.1, J5.1
- net ADC_CLAMP_2V5: now also D201.2 (K), D301.2 (K), D401.2 (K), D501.2 (K), D601.2 (K), D701.2 (K), C24.1, R14.2, R15.1; no longer J16.2, J17.1, J18.1
- net AGND_BUCK: now also U9.24 (AGND), U9.27 (AGND)
- net BATT_RAW: now also F1.3 (RAW), F2.3 (RAW), F3.3 (RAW), F4.3 (RAW), F5.3 (RAW), F6.3 (RAW), F7.3 (RAW), F8.3 (RAW), J2.1 (Pin_1), F10.1; no longer F1.2 (COM), F2.2 (COM), F3.2 (COM), F4.2 (COM), F5.2 (COM), F6.2 (COM), F7.2 (COM), F8.2 (COM), F9.1
- net CC1: now also R7.1; no longer C2.1
- net CC2: now also R8.1; no longer C3.1
- net DEN2: now also R202.1; no longer R204.1
- net DEN3: now also R302.1; no longer R305.1
- net DEN4: now also R402.1; no longer R403.1
- net DEN5: now also R502.1; no longer C503.1
- net DEN6: now also R602.1; no longer D601.1
- net DENR2: now also R202.2, R209.1; no longer D203.1, R204.2
- net DENR3: now also R309.1, R302.2; no longer R305.2
- net DENR4: now also R409.1, R402.2; no longer R403.2
- net DENR5: now also R509.1, R502.2, U5.3 (DEN); no longer C503.2, R501.3 (DEN)
- net DENR6: now also R602.2, R609.1, U6.3 (DEN); no longer D601.2, R602.3 (DEN)
- net DENR7: now also R709.1, U7.3 (DEN); no longer R704.3 (DEN)
- net DENR8: now also R809.1, U8.3 (DEN); no longer R805.3 (DEN)
- net GND: now also C303.2, C503.2, C603.2, D103.1 (A), D103.3 (COM), D201.1 (A), D202.1 (K), D203.1 (A), D203.3 (COM), D301.1 (A), D302.1 (K), D303.1 (A), D303.3 (COM), D401.1 (A), D402.1 (K), D403.1 (A), D403.3 (COM), D5.1 (K), D501.1 (A), D502.1 (K), D503.3 (COM), D601.1 (A), D603.1 (A), D603.3 (COM), D701.1 (A), D703.1 (A), D703.3 (COM), D803.1 (A), D803.3 (COM), J16.2 (Pin_2), J5.1 (Pin_1), R203.2, R204.2, R304.2, R403.2, R503.2, R704.2, U9.16 (PGND), U9.17 (PGND), U9.28 (PGND), U9.29 (PGND), U9.5 (PGND), U9.6 (PGND), C10.2, C201.2, C24.2, C25.2, C26.2, C28.2, C29.2, C301.2, C302.2, C401.2, C402.2, C501.2, C502.2, C601.2, C602.2, C701.2, C702.2, C801.2, C802.2, C9.2, D10.2 (A2), D7.2 (A2), D8.2 (A), J11.2 (Pin_2), J13.2 (Pin_2), R15.2, R29.2, R404.2, R406.2, R504.2, R506.2, R606.2, R7.2, R706.2, R8.2, U15.7 (GND); no longer C204.1 (K), C404.2, C504.2, C604.2, D103.2 (A2), D201.2, D301.2, D302.2, D402.2, D5.2, D501.2, D502.2, D703.2, D803.2, H7.2 (Pin_2), J2.2 (Pin_2), J5.2, R205.2, R207.2, R307.2, R308.1 (K), R407.2, R409.1 (K), R508.2, R608.2, R609.2, R708.2, R709.2, R809.2
- net IN2: now also R201.1; no longer R202.1
- net IN3: now also R301.1; no longer R304.1
- net IN4: now also R401.1; no longer R405.1
- net IN5: now also R501.1; no longer R503.1
- net IN6: now also R601.1; no longer C603.1
- net IN7: now also R701.1; no longer D701.1
- net INR2: now also R208.1, R201.2; no longer R202.2, R209.1
- net INR3: now also R308.1, R301.2; no longer D303.1, R304.2
- net INR4: now also R408.1, R401.2; no longer R405.2
- net INR5: now also R508.1, U5.2 (IN); no longer R503.2
- net INR6: now also R608.1, R601.2, U6.2 (IN); no longer C603.2, R602.2 (IN)
- net INR7: now also R708.1, R701.2, U7.2 (IN); no longer D701.2, R704.2 (IN)
- net INR8: now also U8.2 (IN); no longer R805.2 (IN)
- net IS2: now also C203.1, D201.3 (COM), R205.2; no longer D201.1, R203.2
- net IS3: now also C303.1, D301.3 (COM), R305.2; no longer C303.2
- net IS4: now also C403.1, D401.3 (COM), R405.2; no longer D401.2
- net IS5: now also C503.1, D501.3 (COM)
- net IS6: now also C603.1, D601.3 (COM)
- net IS7: now also D701.3 (COM)
- net IS8: now also R805.2
- net ISP2: now also R204.1; no longer R203.1
- net ISP3: now also R304.1, R305.1; no longer C303.1, R303.1
- net ISP4: now also R405.1, R404.1; no longer C403.1, D401.1
- net ISP5: now also R504.1, U5.4 (IS); no longer D501.1, R501.4 (IS)
- net ISP6: now also U6.4 (IS); no longer R602.4 (IS)
- net ISP7: now also R704.1, U7.4 (IS); no longer R704.4 (IS)
- net ISP8: now also R805.1, U8.4 (IS); no longer R805.4 (IS)
- net LEDK1: now also D103.2 (K)
- net LEDK2: now also D203.2 (K), R207.2; no longer C204.2 (A)
- net LEDK3: now also D302.2 (A), D303.2 (K), R307.2; no longer C304.2, R308.2 (A)
- net LEDK4: now also D402.2 (A), D403.2 (K), R407.2; no longer R408.2, R409.2 (A)
- net LEDK5: now also D502.2 (A), R507.2; no longer R509.2
- net LEDK6: now also R607.2
- net LEDK7: now also D703.2 (K)
- net LEDK8: now also D803.2 (K)
- net LOAD1: now also F1.2 (LOAD), J11.1 (Pin_1); no longer C102.1, F1.3 (LOAD), J2.1 (Pin_1), R106.1, R107.1, U1.10 (OUT), U1.12 (OUT), U1.13 (OUT), U1.14 (OUT), U1.8 (OUT), U1.9 (OUT)
- net LOAD2: now also F2.2 (LOAD); no longer D202.1, F2.3 (LOAD), R206.1, R207.1, U2.10 (OUT), U2.12 (OUT), U2.13 (OUT), U2.14 (OUT), U2.8 (OUT), U2.9 (OUT)
- net LOAD3: now also F3.2 (LOAD), J13.1 (Pin_1); no longer C304.1, D302.1, F3.3 (LOAD), H7.1 (Pin_1), R307.1, U3.10 (OUT), U3.12 (OUT), U3.13 (OUT), U3.14 (OUT), U3.8 (OUT), U3.9 (OUT)
- net LOAD4: now also F4.2 (LOAD); no longer C404.1, D402.1, F4.3 (LOAD), R408.1, U4.10 (OUT), U4.12 (OUT), U4.13 (OUT), U4.14 (OUT), U4.8 (OUT), U4.9 (OUT)
- net LOAD5: now also F5.2 (LOAD); no longer C504.1, F5.3 (LOAD), R501.10 (OUT), R501.12 (OUT), R501.13 (OUT), R501.14 (OUT), R501.8 (OUT), R501.9 (OUT), R508.1, R509.1
- net LOAD6: now also F6.2 (LOAD), J16.1 (Pin_1); no longer D603.1, F6.3 (LOAD), R602.10 (OUT), R602.12 (OUT), R602.13 (OUT), R602.14 (OUT), R602.8 (OUT), R602.9 (OUT), R608.1, R609.1
- net LOAD7: now also F7.2 (LOAD), J17.1 (Pin_1); no longer D703.1, F7.3 (LOAD), R704.10 (OUT), R704.12 (OUT), R704.13 (OUT), R704.14 (OUT), R704.8 (OUT), R704.9 (OUT), R707.1, R709.1
- net LOAD8: now also F8.2 (LOAD), J18.1 (Pin_1); no longer D803.1, F8.3 (LOAD), R805.10 (OUT), R805.12 (OUT), R805.13 (OUT), R805.14 (OUT), R805.8 (OUT), R805.9 (OUT), R806.1, R807.1
- net RT: now also U9.1 (RT)
- net RXD0: now also J5.4 (Pin_4)
- net STATUS_K: now also D5.2 (A)
- net TXD0: now also J5.3 (Pin_3)
- net UGND2: now also C204.2, R203.1; no longer C203.1, D203.2
- net UGND3: now also C304.2, R303.1, R308.2; no longer D301.1, D303.2
- net UGND4: now also C404.2, R403.1, R408.2, R409.2; no longer D403.2
- net UGND5: now also C504.2, R503.1, R508.2, R509.2, U5.1 (GND); no longer R501.1 (GND)
- net UGND6: now also C604.2, R608.2, R609.2, U6.1 (GND); no longer R602.1 (GND)
- net UGND7: now also R708.2, R709.2, U7.1 (GND); no longer R704.1 (GND)
- net UGND8: now also R809.2, U8.1 (GND); no longer R805.1 (GND)
- net USB_D+: now also R10.1; no longer U9.1
- net USB_MCU_D+: now also R10.2; no longer U9.2
- net VCC_BUCK: now also U9.23 (VCC)
- net VIN: now also C2.1, C3.1, U9.18 (VIN), U9.19 (VIN), U9.2 (EN/SYNC), U9.3 (VIN), U9.4 (VIN)
- net VS1 renamed AUTO_PROTECTED
- net AUTO_PROTECTED: now also C204.1, C304.1, C404.1, C504.1, C604.1, C704.1, C804.1, F9.1, U2.15 (VS), U3.15 (VS), U4.15 (VS), C201.1, C29.1, C301.1, C401.1, C501.1, C601.1, C701.1, C801.1, D10.1 (A1), Q10.5 (D), Q11.5 (D), U15.12 (C), U5.15 (VS), U6.15 (VS), U7.15 (VS), U8.15 (VS); no longer D103.1 (A1), F1.1 (SW)
- net VS2 renamed PROFET_OUT2
- net PROFET_OUT2: now also R206.1, R207.1, U2.10 (OUT), U2.12 (OUT), U2.13 (OUT), U2.14 (OUT), U2.8 (OUT), U2.9 (OUT); no longer R208.1, U2.15 (VS)
- net VS3 renamed PROFET_OUT3
- net PROFET_OUT3: now also R307.1, U3.10 (OUT), U3.12 (OUT), U3.13 (OUT), U3.14 (OUT), U3.8 (OUT), U3.9 (OUT), C302.1; no longer R309.1, U3.15 (VS)
- net VS4 renamed PROFET_OUT4
- net PROFET_OUT4: now also U4.10 (OUT), U4.12 (OUT), U4.13 (OUT), U4.14 (OUT), U4.8 (OUT), U4.9 (OUT), C402.1, R406.1; no longer D403.1, U4.15 (VS)
- removed net VS5: D502.1, F5.1 (SW), R501.15 (VS)
- removed net VS6: C604.1, F6.1 (SW), R602.15 (VS)
- removed net VS7: C704.1, F7.1 (SW), R704.15 (VS), R708.1
- removed net VS8: C804.1, F8.1 (SW), R805.15 (VS), R809.1
- new net AUTO_FUSED: C25.1, D6.1 (A1), F10.2, Q6.3 (D), Q7.3 (D), Q8.3 (D), Q9.3 (D), R26.1, R27.1
- new net CAP_AUTO: C27.1, U15.11 (CAP)
- new net DGATE_AUTO: R24.1, R25.1, U15.1 (DGATE)
- new net DGATE_Q10: Q10.4 (G), R24.2
- new net DGATE_Q11: Q11.4 (G), R25.2
- new net HGATE_AUTO: R20.1, R21.1, R22.1, R23.1, U15.8 (HGATE)
- new net HGATE_Q6: Q6.1 (G), R20.2
- new net HGATE_Q7: Q7.1 (G), R21.2
- new net HGATE_Q8: Q8.1 (G), R22.2
- new net HGATE_Q9: Q9.1 (G), R23.2
- new net OV_AUTO: R28.2, R29.1, U15.5 (OV)
- new net OV_DIV_MID: R27.2, R28.1
- new net PROFET_OUT1: C102.1, F1.1 (AUTO), R106.1, R107.1, U1.10 (OUT), U1.12 (OUT), U1.13 (OUT), U1.14 (OUT), U1.8 (OUT), U1.9 (OUT)
- new net PROFET_OUT5: C502.1, F5.1 (AUTO), R506.1, R507.1, U5.10 (OUT), U5.12 (OUT), U5.13 (OUT), U5.14 (OUT), U5.8 (OUT), U5.9 (OUT)
- new net PROFET_OUT6: C602.1, F6.1 (AUTO), R606.1, R607.1, U6.10 (OUT), U6.12 (OUT), U6.13 (OUT), U6.14 (OUT), U6.8 (OUT), U6.9 (OUT)
- new net PROFET_OUT7: C702.1, F7.1 (AUTO), R706.1, R707.1, U7.10 (OUT), U7.12 (OUT), U7.13 (OUT), U7.14 (OUT), U7.8 (OUT), U7.9 (OUT)
- new net PROFET_OUT8: C802.1, F8.1 (AUTO), R806.1, R807.1, U8.10 (OUT), U8.12 (OUT), U8.13 (OUT), U8.14 (OUT), U8.8 (OUT), U8.9 (OUT)
- new net PROTECTION_COMMON_SOURCE: C28.1, D9.2 (A), Q10.1 (S), Q10.2 (S), Q10.3 (S), Q11.1 (S), Q11.2 (S), Q11.3 (S), Q6.2 (S), Q7.2 (S), Q8.2 (S), Q9.2 (S), U15.2 (A), U15.3 (VSNS), U15.4 (SW), U15.9 (OUT)
- new net TVS_INPUT_MID: D6.2 (A2), D7.1 (A1)
- new net VS_CONTROLLER: C26.1, C27.2, D8.1 (K), D9.1 (K), R26.2, U15.10 (VS), U15.6 (EN/UVLO)
Other:
- note added: "AUTO + LOGIC: shared fused LM74800 cutoff. BYPASS: raw battery, no electronics."
- note added: "Channel LEDs indicate PROFET output, not the BYPASS load terminal."
- note added: "ESWITCH — PROTECTION REVISION CANDIDATE / NOT FOR FABRICATION"
- note added: "Recovery: REMOVE F10 to isolate AUTO electronics; move load fuses to BYPASS."
- note added: "SHARED AUTO/LOGIC PROTECTION — BYPASS remains raw battery"
- note removed: "ESWITCH SIMPLE — PROTOTYPE / BENCH QUALIFICATION REQUIRED"
- note removed: "LOGIC: separately fused; no common series switch in branch power paths"
- note removed: "Recovery: all usable channels BYPASS; failed/unused channels fuse REMOVED."
- moved on the sheet: C202, C504, C604, R202, R203, R204, R205, R207, R209, R303, R304, R305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
